File: kicad/neoclock.kicad_pcb (KiCad board)
At the start: 2 copper layers, 41.1 x 42.2 mm, 19 parts, among them CON1 2.1mm 5V, IC1 ATMEGA328P-A, K1 NEOPIXEL, P1 ICSP, P2 FTDI, SW1 HOUR, SW2 MINUTE, U1 DS1307

Commit message: woot
Parts:
- added PHOTOR1: PHOTOR, synic:PHOTORESISTOR, F.Cu at (114.8, 50.8)
- added RV1: BRIGHTNESS, synic:Timmer_Pot_ST32ETA103, F.Cu at (110.2, 56.4)
- added X1: 16Mhz, Crystals:Crystal_HC49-U_Vertical_3Pin, F.Cu at (129.5, 27.9)
- added X2: 32.768kHz, Crystals:Crystal_Round_Horizontal_3mm_BigPad, F.Cu at (121.9, 18.3)
- BT1: footprint Discret:CR2032H -> WANDL:WNL_CR2302_TH_KEYSTONE_3003
- moved C6 30.2 mm to (139.7, 29.0), turned to 90 degrees
- moved C5 26.2 mm to (137.2, 29.0), turned to 90 degrees
- moved C8 24.9 mm to (99.6, 33.5), turned to 180 degrees
- moved C7 14.7 mm to (126.5, 34.0), turned to 0 degrees
- moved C1 13.4 mm to (133.1, 17.3), turned to 180 degrees
- moved C3 12.7 mm to (109.2, 45.2), turned to 90 degrees
- moved C4 10.3 mm to (117.9, 44.2), turned to 90 degrees
- moved IC1 5.92 mm to (132.1, 39.1)
- moved P1 4.68 mm to (138.2, 20.3)
- moved C2 4.34 mm to (136.7, 45.2), turned to 90 degrees
- moved U1 3.70 mm to (127.5, 21.8)
- moved D1 3.09 mm to (126.5, 17.3)
- moved SW2 3.05 mm to (135.6, 56.4)
- moved K1 3.05 mm to (104.1, 17.8)
- moved P2 3.05 mm to (98.6, 23.9)
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Routing:
- net GND: track 123.1 -> 16.8 mm, vias 5 -> 3
- net BRIGHTNESS: track 0.00 -> 45.9 mm, vias 0 -> 2
- net Net-(IC1-Pad26): track 0.00 -> 32.7 mm, vias 0 -> 2
- net Net-(C5-Pad2): track 0.00 -> 30.3 mm, vias 0 -> 1
- net Net-(C6-Pad2): track 8.22 -> 35.8 mm, vias 0 -> 1
- net I2CSCL: track 0.00 -> 23.1 mm, vias 0 -> 2
- net VCC: track 100.4 -> 121.0 mm
- net Net-(C2-Pad1): track 14.1 -> 0.00 mm, vias 2 -> 0
- net I2CSDA: track 0.00 -> 12.9 mm, vias 0 -> 2
- net Net-(IC1-Pad2): track 22.7 -> 33.1 mm, vias 1 -> 3
- net Net-(IC1-Pad9): track 41.9 -> 32.7 mm
- net Net-(IC1-Pad1): track 24.0 -> 30.1 mm
- net Net-(BT1-Pad1): track 31.0 -> 36.5 mm, vias 1 -> 0
- net Net-(U1-Pad2): track 0.00 -> 4.91 mm
- net Net-(U1-Pad1): track 0.00 -> 3.89 mm
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- added copper zone on F.Cu, net GND
- removed copper zone on F.Cu, net VCC
Other:
- board size 41.1 x 42.2 mm -> 45.2 x 45.2 mm

Commit message: woo
Parts:
- BT1: footprint WANDL:WNL_CR2302_TH_KEYSTONE_3003 -> WNL_CR2302_TH_KEYSTONE_3003
Routing:
- net Net-(C8-Pad2): track 0.00 -> 50.9 mm, vias 0 -> 4
- net FTDI3: track 0.00 -> 43.3 mm, vias 0 -> 2
- net FTDI2: track 0.00 -> 41.5 mm, vias 0 -> 1
- net VCC: track 121.0 -> 137.7 mm
- net GND: track 16.8 -> 19.8 mm
- net Net-(IC1-Pad1): track 30.1 -> 28.4 mm
- net Net-(IC1-Pad10): track 43.7 -> 42.9 mm

Commit message: woot
Parts:
- added R1: 330, Resistors_SMD:Resistor_SMD0805_HandSoldering, F.Cu at (102.9, 24.1)
- added R2: 10k, Resistors_SMD:Resistor_SMD0805_HandSoldering, F.Cu at (138.3, 37.8)
- added R3: 10k, Resistors_SMD:Resistor_SMD0805_HandSoldering, F.Cu at (121.5, 17.9)
- BT1: moved to B.Cu
- RV1: value BRIGHTNESS -> POT
- moved RV1 43.3 mm to (131.2, 18.5), turned to 90 degrees
- moved X2 27.1 mm to (106.6, 40.6), turned to 270 degrees
- moved D1 23.4 mm to (103.1, 17.5), turned to 180 degrees
- moved K1 22.1 mm to (98.6, 39.1), turned to 90 degrees
- moved C1 19.7 mm to (118.2, 30.2), turned to 90 degrees
- moved U1 17.4 mm to (112.1, 30.0)
- moved JP1 14.3 mm to (111.9, 44.2), turned to 180 degrees
- moved C5 10.9 mm to (128.0, 23.1)
- moved C3 10.6 mm to (110.2, 55.8), turned to 270 degrees
- moved C6 10.3 mm to (131.2, 23.1)
- moved PHOTOR1 7.30 mm to (116.5, 57.9)
- moved C4 4.97 mm to (117.5, 49.1)
- moved C2 4.46 mm to (138.2, 49.4), turned to 0 degrees
- moved IC1 4.10 mm to (130.9, 43.1)
- moved C7 3.31 mm to (124.7, 36.8)
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Connections:
- BT1 pad 2: (no net) -> GND
Routing:
- net VCC: track 137.7 -> 225.4 mm, vias 1 -> 0
- net GND: track 19.8 -> 99.7 mm, vias 3 -> 9
- net Net-(IC1-Pad26): track 32.7 -> 102.0 mm, vias 2 -> 1
- net Net-(C8-Pad2): track 50.9 -> 93.0 mm, vias 4 -> 0
- net Net-(IC1-Pad17): track 0.00 -> 31.8 mm, vias 0 -> 1
- net Net-(IC1-Pad15): track 0.00 -> 29.7 mm, vias 0 -> 1
- net Net-(IC1-Pad16): track 0.00 -> 28.3 mm, vias 0 -> 1
- net BRIGHTNESS: track 45.9 -> 21.4 mm, vias 2 -> 0
- net Net-(IC1-Pad9): track 32.7 -> 18.5 mm
- net Net-(U1-Pad1): track 3.89 -> 16.6 mm
- net Net-(C2-Pad1): track 0.00 -> 11.1 mm, vias 0 -> 2
- net Net-(IC1-Pad2): track 33.1 -> 23.0 mm, vias 3 -> 1
- net Net-(C6-Pad2): track 35.8 -> 26.2 mm
- net I2CSDA: track 12.9 -> 22.4 mm
- net Net-(U1-Pad2): track 4.91 -> 13.4 mm
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Other:
- outline, holes or cut-outs redrawn
- board text added: "NeoClock arolsen@gmail.com"

Commit message: updating clock board
Parts:
- BT1: footprint WNL_CR2302_TH_KEYSTONE_3003 -> WANDL:WNL_CR2302_TH_KEYSTONE_3003; moved to F.Cu
- JP1, K1: footprint Connect:SIL-3 -> Pin_Headers:Pin_Header_Straight_1x03
- P2: footprint Connect:SIL-6 -> Pin_Headers:Pin_Header_Straight_1x06
- PHOTOR1: footprint synic:PHOTORESISTOR -> PHOTORESISTOR
- SW1, SW2: footprint Discret:SW_PUSH_SMALL -> synic:SW_PUSH_SMALL
- X1: footprint Crystals:Crystal_HC49-U_Vertical_3Pin -> synic:Crystal_HC49-SMALL_SMD
- X2: footprint Crystals:Crystal_Round_Horizontal_3mm_BigPad -> Crystal-4pad
- moved C6 95.5 mm to (87.4, 108.0), turned to 0 degrees
- moved X1 92.7 mm to (76.2, 105.2)
- moved R2 91.5 mm to (62.2, 88.8), turned to 0 degrees
- moved P2 91.5 mm to (90.9, 115.1), turned to 0 degrees
- moved SW2 84.9 mm to (77.9, 118.6)
- moved C5 83.0 mm to (90.7, 97.3), turned to 0 degrees
- moved JP1 81.0 mm to (68.5, 112.5), turned to 0 degrees
- moved R1 80.0 mm to (111.0, 103.8)
- moved R3 79.8 mm to (95.2, 93.2)
- moved K1 75.7 mm to (52.3, 99.1), turned to 0 degrees
- moved C2 74.5 mm to (82.0, 98.4)
- moved IC1 69.3 mm to (61.7, 47.2)
- moved RV1 68.9 mm to (74.9, 58.3), turned to 0 degrees
- moved C1 68.1 mm to (77.1, 84.5), turned to 0 degrees
- moved P1 63.7 mm to (93.0, 64.8), turned to 0 degrees
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Routing:
- net VCC: track 225.4 -> 0.00 mm
- net Net-(IC1-Pad26): track 102.0 -> 0.00 mm, vias 1 -> 0
- net GND: track 99.7 -> 0.00 mm, vias 9 -> 0
- net Net-(C8-Pad2): track 93.0 -> 0.00 mm
- net FTDI3: track 38.5 -> 0.00 mm
- net FTDI2: track 37.9 -> 0.00 mm, vias 1 -> 0
- net Net-(IC1-Pad10): track 37.0 -> 0.00 mm, vias 1 -> 0
- net Net-(BT1-Pad1): track 35.5 -> 0.00 mm
- net Net-(IC1-Pad17): track 31.8 -> 0.00 mm, vias 1 -> 0
- net Net-(IC1-Pad15): track 29.7 -> 0.00 mm, vias 1 -> 0
- net Net-(IC1-Pad16): track 28.3 -> 0.00 mm, vias 1 -> 0
- net Net-(C6-Pad2): track 26.2 -> 0.00 mm, vias 1 -> 0
- net Net-(IC1-Pad1): track 25.6 -> 0.00 mm, vias 1 -> 0
- net Net-(C5-Pad2): track 25.3 -> 0.00 mm, vias 1 -> 0
- net Net-(IC1-Pad2): track 23.0 -> 0.00 mm, vias 1 -> 0
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- removed copper zone on B.Cu, net GND
- removed copper zone on F.Cu, net GND
Other:
- board size 45.2 x 45.2 mm -> 101.4 x 101.4 mm
- board text removed: "NeoClock arolsen@gmail.com"

Commit message: updates
Parts:
- BT1: footprint WANDL:WNL_CR2302_TH_KEYSTONE_3003 -> synic:WNL_CR2302_TH_KEYSTONE_3003
- moved SW1 100.5 mm to (26.4, 49.0), turned to 270 degrees
- moved CON1 97.5 mm to (29.5, 28.1)
- moved SW2 94.1 mm to (26.4, 39.9), turned to 270 degrees
- moved R1 91.7 mm to (32.8, 55.9), turned to 90 degrees
- moved JP1 88.6 mm to (53.8, 25.1), turned to 180 degrees
- moved C6 81.7 mm to (32.8, 47.2), turned to 90 degrees
- moved C5 79.1 mm to (32.8, 43.4), turned to 90 degrees
- moved P2 74.4 mm to (38.1, 62.7)
- moved K1 74.3 mm to (45.2, 25.1)
- moved R3 73.9 mm to (52.3, 33.0), turned to 90 degrees
- moved C7 73.2 mm to (45.7, 51.8), turned to 90 degrees
- moved C8 72.9 mm to (48.0, 35.3), turned to 180 degrees
- moved X1 71.5 mm to (36.8, 45.5), turned to 270 degrees
- moved P1 67.1 mm to (25.9, 61.5), turned to 180 degrees
- moved R2 56.2 mm to (55.4, 33.0), turned to 270 degrees
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Routing:
- net VCC: track 0.00 -> 167.8 mm
- net GND: track 0.00 -> 153.1 mm, vias 0 -> 11
- net Net-(C8-Pad2): track 0.00 -> 74.5 mm
- net Net-(BT1-Pad1): track 0.00 -> 52.8 mm
- net Net-(IC1-Pad17): track 0.00 -> 47.1 mm, vias 0 -> 2
- net Net-(IC1-Pad16): track 0.00 -> 37.3 mm, vias 0 -> 1
- net Net-(IC1-Pad15): track 0.00 -> 35.5 mm, vias 0 -> 2
- net Net-(C8-Pad1): track 0.00 -> 34.6 mm, vias 0 -> 1
- net Net-(IC1-Pad10): track 0.00 -> 32.4 mm, vias 0 -> 1
- net Net-(IC1-Pad9): track 0.00 -> 30.7 mm, vias 0 -> 1
- net FTDI2: track 0.00 -> 28.4 mm, vias 0 -> 1
- net FTDI3: track 0.00 -> 27.9 mm, vias 0 -> 1
- net Net-(U1-Pad1): track 0.00 -> 26.3 mm
- net Net-(IC1-Pad2): track 0.00 -> 25.7 mm, vias 0 -> 1
- net Net-(IC1-Pad1): track 0.00 -> 24.8 mm, vias 0 -> 1
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- added copper zone on B.Cu, net GND
- added copper zone on F.Cu, net GND
Other:
- board size 101.4 x 101.4 mm -> 64.8 x 41.9 mm
- rule trace_min: 0.254 -> 0.2
- board text added: "NeoClock v0 by Adam Olsen arolsen@gmail.com"

Commit message: woot
Parts:
- K1: footprint Pin_Headers:Pin_Header_Straight_1x03 -> jst-3-pth-ra
- moved PHOTOR1 47.4 mm to (25.1, 55.9), turned to 0 degrees
- moved RV1 28.8 mm to (50.8, 59.4), turned to 0 degrees
- moved D1 22.3 mm to (26.4, 33.8), turned to 180 degrees
- moved C8 16.5 mm to (45.0, 51.6), turned to 0 degrees
- moved R1 11.7 mm to (32.3, 44.2)
- moved C5 11.2 mm to (32.5, 54.6), turned to 180 degrees
- moved C7 9.45 mm to (40.1, 44.2)
- moved C6 8.29 mm to (36.6, 54.6), turned to 0 degrees
- moved C3 7.26 mm to (36.8, 37.6)
- moved BT1 6.10 mm to (68.3, 36.3)
- moved X1 4.60 mm to (36.3, 50.0), turned to 0 degrees
- moved K1 4.33 mm to (45.5, 29.5)
- moved C4 2.74 mm to (43.2, 36.8)
- moved C1 0.72 mm to (57.4, 58.9)
- moved P1 0.25 mm to (25.9, 61.7)
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Routing:
- net Net-(IC1-Pad26): track 23.9 -> 103.6 mm, vias 0 -> 1
- net Net-(C8-Pad2): track 74.5 -> 139.6 mm, vias 0 -> 1
- net GND: track 153.1 -> 99.0 mm, vias 11 -> 6
- net Net-(BT1-Pad1): track 52.8 -> 35.3 mm
- net Net-(C8-Pad1): track 34.6 -> 20.4 mm
- net BRIGHTNESS: track 11.4 -> 21.6 mm, vias 0 -> 2
- net Net-(IC1-Pad10): track 32.4 -> 22.8 mm
- net Net-(IC1-Pad16): track 37.3 -> 30.9 mm, vias 1 -> 0
- net Net-(IC1-Pad17): track 47.1 -> 41.5 mm, vias 2 -> 0
- net VCC: track 167.8 -> 170.9 mm
- net Net-(IC1-Pad9): track 30.7 -> 33.5 mm
- net Net-(IC1-Pad15): track 35.5 -> 37.9 mm, vias 2 -> 0
- net Net-(C2-Pad1): track 8.08 -> 10.0 mm
- net Net-(D1-Pad1): track 10.1 -> 11.7 mm
- net FTDI2: track 28.4 -> 29.5 mm
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Other:
- board size 64.8 x 41.9 mm -> 58.2 x 41.9 mm
- net class VCC added: clearance 0.254, trace_width 0.3, via_dia 0.889, via_drill 0.635

Commit message: updating pcb finally
Parts:
- removed C8: 100nF, Capacitors_SMD:c_0805
- removed JP1: AUTOBRGT, Pin_Headers:Pin_Header_Straight_1x03
- removed P2: FTDI, Pin_Headers:Pin_Header_Straight_1x06
- removed RV1: POT, synic:Timmer_Pot_ST32ETA103
- BT1: footprint synic:WNL_CR2302_TH_KEYSTONE_3003 -> synic:BK-755_12mm_coincell
- CON1: footprint Connect:BARREL_JACK -> synic:BARREL_JACK_SMD
- K1: footprint jst-3-pth-ra -> synic:jst-3-pth-ra
- PHOTOR1: footprint PHOTORESISTOR -> synic:PHOTORESISTOR
- SW1, SW2: footprint synic:SW_PUSH_SMALL -> synic:SMD_PUSHBUTTON_MINI
- U1: footprint SOIC8:Test -> SOIC_Packages:SOIC-8_N
- X1: footprint synic:Crystal_HC49-SMALL_SMD -> synic:4padCrystalSMD_7.0x5.0mm
- X2: footprint Crystal-4pad -> synic:4padCrystalSMD_7.0x5.0mm
- moved X2 39.9 mm to (34.3, 57.0), turned to 0 degrees
- moved BT1 39.8 mm to (34.3, 57.0), turned to 0 degrees
- moved R2 32.0 mm to (34.3, 57.0), turned to 0 degrees
- moved U1 30.5 mm to (34.3, 57.0)
- moved R3 30.0 mm to (34.3, 57.0), turned to 0 degrees
- moved K1 29.8 mm to (34.3, 57.0)
- moved CON1 29.4 mm to (34.3, 57.0)
- moved D1 24.6 mm to (34.3, 57.0), turned to 0 degrees
- moved C2 23.7 mm to (34.3, 57.0), turned to 0 degrees
- moved C1 23.2 mm to (34.3, 57.0), turned to 0 degrees
- moved C4 22.1 mm to (34.3, 57.0), turned to 0 degrees
- moved IC1 20.8 mm to (34.3, 57.0)
- moved C3 19.6 mm to (34.3, 57.0)
- moved SW2 18.9 mm to (34.3, 57.0), turned to 0 degrees
- moved C7 14.1 mm to (34.3, 57.0), turned to 0 degrees
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Connections:
- IC1 pad 25: BRIGHTNESS -> Net-(IC1-Pad25)
Routing:
- net VCC: track 170.9 -> 0.00 mm
- net Net-(IC1-Pad29): track 139.6 -> 0.00 mm, vias 1 -> 0
- net Net-(IC1-Pad26): track 103.6 -> 0.00 mm, vias 1 -> 0
- net GND: track 99.0 -> 0.00 mm, vias 6 -> 0
- net Net-(IC1-Pad17): track 41.5 -> 0.00 mm
- net Net-(IC1-Pad15): track 37.9 -> 0.00 mm
- net Net-(BT1-Pad1): track 35.3 -> 0.00 mm
- net Net-(IC1-Pad9): track 33.5 -> 0.00 mm, vias 1 -> 0
- net Net-(IC1-Pad16): track 30.9 -> 0.00 mm
- net FTDI2: track 29.5 -> 0.00 mm, vias 1 -> 0
- net FTDI3: track 27.9 -> 0.00 mm, vias 1 -> 0
- net Net-(U1-Pad1): track 26.3 -> 0.00 mm
- net Net-(IC1-Pad2): track 25.7 -> 0.00 mm, vias 1 -> 0
- net Net-(IC1-Pad1): track 24.8 -> 0.00 mm, vias 1 -> 0
- net Net-(IC1-Pad10): track 22.8 -> 0.00 mm, vias 1 -> 0
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- removed copper zone on B.Cu, net GND
- removed copper zone on F.Cu, net GND
Other:
- board size 58.2 x 41.9 mm -> 30.5 x 30.5 mm
- net class VCC removed
- rule trace_min: 0.2 -> 0.254
- board text removed: "NeoClock v0 by Adam Olsen arolsen@gmail.com"

Commit message: woot
Parts:
- BT1: moved to B.Cu
- X1: footprint synic:4padCrystalSMD_7.0x5.0mm -> synic:2_SMD_CRYSTAL_5.0x3.20
- X2: footprint synic:4padCrystalSMD_7.0x5.0mm -> synic:2_SMD_CRYSTAL_3.2x1.5
- moved U1 39.0 mm to (23.1, 19.7), turned to 90 degrees
- moved PHOTOR1 38.5 mm to (32.5, 18.5), turned to 180 degrees
- moved R1 37.7 mm to (37.2, 19.4), turned to 270 degrees
- moved K1 35.1 mm to (42.7, 23.0)
- moved X2 34.5 mm to (31.9, 22.6), turned to 270 degrees
- moved C7 33.4 mm to (25.7, 24.8)
- moved R2 32.2 mm to (21.8, 27.3)
- moved D1 31.9 mm to (45.8, 27.3), turned to 270 degrees
- moved C2 31.1 mm to (40.4, 26.5)
- moved C5 29.8 mm to (21.5, 30.1)
- moved IC1 25.7 mm to (33.7, 31.4)
- moved X1 25.5 mm to (21.1, 35.2), turned to 270 degrees
- moved C1 21.4 mm to (27.3, 36.8), turned to 180 degrees
- moved C6 21.0 mm to (21.5, 40.4)
- moved C4 20.9 mm to (40.9, 37.2)
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Routing:
- net VCC: track 0.00 -> 83.6 mm, vias 0 -> 2
Other:
- board size 30.5 x 30.5 mm -> 28.1 x 42.7 mm
- net class POWER added: clearance 0.254, trace_width 0.35, via_dia 0.889, via_drill 0.635
- board text added: "+"
