File: kicad/neoclock.kicad_pcb (KiCad board)
At the start: 2 copper layers, 31 x 39.6 mm, 28 parts, among them CON1 1.2mm 5v, K1 NEO, P1 TC2030-CTX, P2 PHOTOR, SW1 HOUR, SW2 MINUTE, SW3 HOUR, SW4 MINUTE, U1 stm32f303x, U2 TLV702xx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

Commit message: board is done?
Parts:
- moved C3 10.1 mm to (45.9, 59.6), turned to 90 degrees
- moved R2 4.38 mm to (44.5, 64.8), turned to 0 degrees
- moved R3 3.30 mm to (42.0, 64.9), turned to 180 degrees
- moved MH1 0.28 mm to (41.8, 60.7)
- moved MH 0.25 mm to (58.2, 50.3)
- moved SW1 0.14 mm to (37.7, 64.9)
- moved SW2 0.09 mm to (37.7, 71.1)
Routing:
- net GND: track 90.0 -> 154.9 mm, vias 6 -> 11
- net VDD: track 83.0 -> 117.5 mm, vias 0 -> 2
- net Net-(K1-Pad3): track 22.9 -> 35.6 mm, vias 1 -> 3
- net Net-(BT1-Pad1): track 45.0 -> 33.2 mm
- net VCC5V: track 43.6 -> 53.4 mm, vias 0 -> 2
- net Net-(R1-Pad1): track 0.00 -> 4.81 mm, vias 0 -> 2
- net Net-(SW2-Pad1): track 29.5 -> 32.9 mm, vias 3 -> 2
- net Net-(R4-Pad1): track 5.65 -> 7.55 mm, vias 0 -> 2
- net NRST: track 29.6 -> 30.6 mm, vias 3 -> 2
- net Net-(P2-Pad1): track 12.4 -> 13.4 mm, vias 2 -> 0
- net SWCLK: track 28.7 -> 29.6 mm
- net Net-(SW1-Pad1): track 33.4 -> 34.2 mm
- net SWDIO: track 20.0 -> 20.8 mm
- added copper zone on B.Cu, net GND
- added copper zone on F.Cu, net GND
Other:
- board text added: "NeoClock v7.0 arolsen@gmail.com"

Commit message: wooters
Parts:
- removed MH, MH1: MountingHole_2-5mm_RevA_Date21Jun2010, Mounting_Holes:MountingHole_2-5mm
- removed SW3: HOUR, synic:KMR2_MICROMINIATURE_BUTTON
- removed SW4: MINUTE, synic:KMR2_MICROMINIATURE_BUTTON
- added C11: 100nF, Capacitors_SMD:C_0805, F.Cu at (43.8, 56.4)
- added C4: 100nF, Capacitors_SMD:C_0805, F.Cu at (43.2, 63.1)
- added D1: RED, LEDs:LED-0805, F.Cu at (39.7, 70.4)
- added D2: GREEN, LEDs:LED-0805, F.Cu at (41.6, 70.4)
- added R5: 330, Resistors_SMD:R_0805, F.Cu at (34.0, 70.4)
- added R6: 330, Resistors_SMD:R_0805, F.Cu at (36.3, 70.4)
- added U3: TXS0101, SMD_Packages:SOT-23-6, F.Cu at (43.1, 59.8)
- added U4: NEO, synicpretty:TESTPOINT, B.Cu at (61.0, 46.2)
- added U5: GND, synicpretty:TESTPOINT, B.Cu at (33.1, 48.0)
- added U6: VCC5V, synicpretty:TESTPOINT, B.Cu at (32.8, 36.1)
- C5, C6, C7, C8: footprint Capacitors_SMD:C_0603 -> Capacitors_SMD:C_0805
- R1, R2, R3, R4: footprint Resistors_SMD:R_0603 -> Resistors_SMD:R_0805
- SW1, SW2: footprint synic:jst-2-pth-ra -> synic:KMR2_MICROMINIATURE_BUTTON
- moved C3 21.3 mm to (56.6, 41.2), turned to 0 degrees
- moved R1 16.3 mm to (36.1, 51.4), turned to 90 degrees
- moved R3 16.0 mm to (33.5, 51.4), turned to 90 degrees
- moved C8 14.9 mm to (59.9, 53.1)
- moved C7 14.5 mm to (59.4, 62.7)
- moved SW2 13.0 mm to (50.7, 70.4)
- moved C5 11.2 mm to (47.8, 63.1), turned to 180 degrees
- moved C2 11.0 mm to (50.3, 48.5), turned to 0 degrees
- moved SW1 10.8 mm to (46.9, 70.4)
- moved P2 10.0 mm to (33.2, 65.2), turned to 270 degrees
- moved X1 9.46 mm to (54.8, 50.9), turned to 180 degrees
- moved C6 9.12 mm to (50.3, 50.7), turned to 0 degrees
- moved C1 6.89 mm to (58.3, 47.3), turned to 180 degrees
- moved R2 5.56 mm to (43.9, 70.4), turned to 270 degrees
- moved K1 3.94 mm to (37.6, 57.8)
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Connections:
- R1 pad 2: GND -> VDD
- R2 pad 2: GND -> VDD
- U1 pad 31: Net-(K1-Pad3) -> Net-(U1-Pad31)
Routing:
- net Net-(P2-Pad1): track 13.4 -> 44.5 mm, vias 0 -> 1
- net GND: track 154.9 -> 181.4 mm, vias 11 -> 7
- net SWCLK: track 29.6 -> 7.71 mm
- net Net-(R1-Pad1): track 4.81 -> 24.5 mm
- net Net-(D1-Pad1): track 0.00 -> 17.5 mm, vias 0 -> 2
- net Net-(D2-Pad1): track 0.00 -> 15.2 mm, vias 0 -> 2
- net Net-(U1-Pad31): track 0.00 -> 15.1 mm, vias 0 -> 2
- net NRST: track 30.6 -> 45.5 mm
- net Net-(SW1-Pad1): track 34.2 -> 23.7 mm
- net SWDIO: track 20.8 -> 12.5 mm
- net Net-(SW2-Pad1): track 32.9 -> 24.9 mm
- net VCC5V: track 53.4 -> 60.9 mm
- net Net-(D2-Pad2): track 0.00 -> 6.95 mm
- net Net-(D1-Pad2): track 0.00 -> 6.36 mm
- net Net-(CON1-Pad1): track 12.7 -> 19.0 mm, vias 0 -> 1
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Other:
- board text added: "NeoClock v8 arolsen@gmail.com"
- board text removed: "NeoClock v7.0 arolsen@gmail.com"

Commit message: bleh
Connections:
- U3 pad 5: VCC5V -> VDD
Routing:
- net VDD: track 115.1 -> 121.9 mm
- net VCC5V: track 60.9 -> 59.0 mm
- net GND: track 181.4 -> 180.3 mm
