File: kicad/neoclock.sch (KiCad schematic (older format))
At the start: 18 parts

Commit message: yeah
Parts:
- added JP1: AUTOBRGT, symbol JUMPER3
- added PHOTOR1: PHOTOR, symbol PHOTOR
- added R3: 10k, symbol R
- added RV1: POT, symbol POT
- added SW1: HOUR, symbol SW_PUSH
- added SW2: MINUTE, symbol SW_PUSH
- gave numbers to parts that had none: 18
Connections:
- net labels added: BRIGHTNESS
- wire segments 64 -> 88
- no-connect marks 11 -> 12

Commit message: added pcb start
Parts:
- added C8: 100nF, symbol C
- added P2: FTDI, symbol CONN_6
Connections:
- net labels added: FTDI2, FTDI3
- wire segments 88 -> 96
Changed lines of the file:
@@
 	5500 1350 5500 2800
 Wire Wire Line
-	5500 2800 3500 2800
-Wire Wire Line
-	3500 2800 3500 2700
+	3500 2800 6600 2800
+Wire Wire Line
+	3500 2700 3500 2800
 Connection ~ 3500 2700
 $Comp
@@
 Wire Wire Line
 	5850 3150 5850 3250
-NoConn ~ 3450 2850
 NoConn ~ 3450 2950
 NoConn ~ 3450 3050
@@
 	750  2100 850  2100
 Connection ~ 850  2100
+$Comp
+L CONN_6 P2
+U 1 1 53444226
+P 7400 4400
+F 0 "P2" V 7350 4400 60  0000 C CNN
+F 1 "FTDI" V 7450 4400 60  0000 C CNN
+F 2 "" H 7400 4400 60  0000 C CNN
+F 3 "" H 7400 4400 60  0000 C CNN
+	1    7400 4400
+	0    -1   1    0
+$EndComp
+Text GLabel 3800 2850 2    60   BiDi ~ 0
+FTDI3
+Wire Wire Line
+	3450 2850 3800 2850
+Text GLabel 7350 3900 1    60   BiDi ~ 0
+FTDI3
+Wire Wire Line
+	7350 4050 7350 3900
+Text GLabel 7250 3900 1    60   BiDi ~ 0
+FTDI2
+Wire Wire Line
+	7250 3900 7250 4050
+Text GLabel 3800 2950 2    60   BiDi ~ 0
+FTDI2
+Wire Wire Line
+	3800 2950 3450 2950
+$Comp
+L C C8
+U 1 1 534444CA
+P 6800 4050
+F 0 "C8" H 6800 4150 40  0000 L CNN
+F 1 "100nF" H 6806 3965 40  0000 L CNN
+F 2 "" H 6838 3900 30  0000 C CNN
+F 3 "" H 6800 4050 60  0000 C CNN
+	1    6800 4050
+	0    1    1    0
+$EndComp
+Wire Wire Line
+	7150 4050 7000 4050
+Wire Wire Line
+	6600 2800 6600 4050
+Connection ~ 5500 2800
+$Comp
+L GND #PWR031
+U 1 1 534445B7
+P 7650 3850
+F 0 "#PWR031" H 7650 3850 30  0001 C CNN
+F 1 "GND" H 7650 3780 30  0001 C CNN
+F 2 "" H 7650 3850 60  0000 C CNN
+F 3 "" H 7650 3850 60  0000 C CNN
+	1    7650 3850
+	-1   0    0    1
+$EndComp
+Wire Wire Line
+	7650 3850 7650 4050
+$Comp
+L VCC #PWR032
+U 1 1 53444635
+P 7450 3850
+F 0 "#PWR032" H 7450 3950 30  0001 C CNN
+F 1 "VCC" H 7450 3950 30  0000 C CNN
+F 2 "" H 7450 3850 60  0000 C CNN
+F 3 "" H 7450 3850 60  0000 C CNN
+	1    7450 3850
+	1    0    0    -1
+$EndComp
+Wire Wire Line
+	7450 3850 7450 4050
+NoConn ~ 7550 4050
 $EndSCHEMATC

Commit message: woot
Connections:
- wire segments 96 -> 110
Changed lines of the file:
@@
 $EndComp
 Wire Wire Line
-	1550 3350 1550 3650
+	1550 3350 1550 3450
+Wire Wire Line
+	1550 3450 1550 3550
+Wire Wire Line
+	1550 3550 1550 3650
 Connection ~ 1550 3450
 Connection ~ 1550 3550
@@
 Connection ~ 1550 3350
 Wire Wire Line
-	1550 1250 1550 1550
+	1550 1250 1550 1350
+Wire Wire Line
+	1550 1350 1550 1550
 Connection ~ 1550 1550
 Connection ~ 1550 1350
@@
 	3800 1850 3800 1600
 Wire Wire Line
-	3800 1600 4300 1600
+	3800 1600 4100 1600
+Wire Wire Line
+	4100 1600 4300 1600
 Connection ~ 4100 1600
 Wire Wire Line
-	3800 2200 4300 2200
+	3800 2200 4100 2200
+Wire Wire Line
+	4100 2200 4300 2200
 Wire Wire Line
 	3450 1950 3800 1950
@@
 	9600 1950 9900 1950
 Wire Wire Line
-	10500 1950 10600 1950
+	10500 1950 10550 1950
+Wire Wire Line
+	10550 1950 10600 1950
 $Comp
 L VCC #PWR011
@@
 $EndComp
 Wire Wire Line
-	3700 850  3700 1150
+	3700 850  3700 950
+Wire Wire Line
+	3700 950  3700 1150
 $Comp
 L CP1 C3
@@
 $EndComp
 Wire Wire Line
-	3700 750  4750 750
+	3700 750  4050 750
+Wire Wire Line
+	4050 750  4400 750
+Wire Wire Line
+	4400 750  4750 750
 Connection ~ 4050 750
 Wire Wire Line
-	3700 1150 4750 1150
+	3700 1150 4050 1150
+Wire Wire Line
+	4050 1150 4400 1150
+Wire Wire Line
+	4400 1150 4750 1150
 Connection ~ 3700 950
 Connection ~ 4050 1150
@@
 	5500 1350 5500 2800
 Wire Wire Line
-	3500 2800 6600 2800
+	3500 2800 5500 2800
+Wire Wire Line
+	5500 2800 6600 2800
 Wire Wire Line
 	3500 2700 3500 2800
@@
 	5200 1650 5200 1750
 Wire Wire Line
-	5200 2250 5200 2550
+	5200 2250 5200 2400
+Wire Wire Line
+	5200 2400 5200 2550
 Wire Wire Line
 	4600 2550 4700 2550
@@
 	3450 3350 3650 3350
 Wire Wire Line
-	3650 3300 3650 3400
+	3650 3300 3650 3350
+Wire Wire Line
+	3650 3350 3650 3400
 Wire Wire Line
 	3650 3400 3900 3400

Commit message: updating pcb finally
Parts:
- removed C8: 100nF, symbol C
- removed JP1: AUTOBRGT, symbol JUMPER3
- removed P2: FTDI, symbol CONN_6
- removed RV1: POT, symbol POT
Connections:
- net labels removed: BRIGHTNESS
- wire segments 110 -> 82
- no-connect marks 12 -> 13
Changed lines of the file:
@@
 LIBS:ds1307timer
 LIBS:open-project
-LIBS:neoclock-cache
 EELAYER 24 0
 EELAYER END
@@
 $EndComp
 Wire Wire Line
-	1550 3350 1550 3450
-Wire Wire Line
-	1550 3450 1550 3550
-Wire Wire Line
-	1550 3550 1550 3650
+	1550 3350 1550 3650
 Connection ~ 1550 3450
 Connection ~ 1550 3550
@@
 Connection ~ 1550 3350
 Wire Wire Line
-	1550 1250 1550 1350
-Wire Wire Line
-	1550 1350 1550 1550
+	1550 1250 1550 1550
 Connection ~ 1550 1550
 Connection ~ 1550 1350
@@
 	3800 1850 3800 1600
 Wire Wire Line
-	3800 1600 4100 1600
-Wire Wire Line
-	4100 1600 4300 1600
+	3800 1600 4300 1600
 Connection ~ 4100 1600
 Wire Wire Line
-	3800 2200 4100 2200
-Wire Wire Line
-	4100 2200 4300 2200
+	3800 2200 4300 2200
 Wire Wire Line
 	3450 1950 3800 1950
@@
 	4700 1600 4750 1600
 $Comp
-L DS1307 U1
-U 1 1 53435651
-P 8500 2500
-F 0 "U1" H 8600 1300 60  0000 C CNN
-F 1 "DS1307" H 8500 2550 60  0000 C CNN
-F 2 "" H 8500 2500 60  0000 C CNN
-F 3 "" H 8500 2500 60  0000 C CNN
-	1    8500 2500
-	1    0    0    -1
-$EndComp
-$Comp
 L VCC #PWR08
 U 1 1 53435693
@@
 	9600 1950 9900 1950
 Wire Wire Line
-	10500 1950 10550 1950
-Wire Wire Line
-	10550 1950 10600 1950
+	10500 1950 10600 1950
 $Comp
 L VCC #PWR011
@@
 $EndComp
 Wire Wire Line
-	3700 850  3700 950
-Wire Wire Line
-	3700 950  3700 1150
+	3700 850  3700 1150
 $Comp
 L CP1 C3
@@
 $EndComp
 Wire Wire Line
-	3700 750  4050 750
-Wire Wire Line
-	4050 750  4400 750
-Wire Wire Line
-	4400 750  4750 750
+	3700 750  4750 750
 Connection ~ 4050 750
 Wire Wire Line
-	3700 1150 4050 1150
-Wire Wire Line
-	4050 1150 4400 1150
-Wire Wire Line
-	4400 1150 4750 1150
+	3700 1150 4750 1150
 Connection ~ 3700 950
 Connection ~ 4050 1150
@@
 	5500 1350 5500 2800
 Wire Wire Line
-	3500 2800 5500 2800
-Wire Wire Line
-	5500 2800 6600 2800
-Wire Wire Line
-	3500 2700 3500 2800
+	5500 2800 3500 2800
+Wire Wire Line
+	3500 2800 3500 2700
 Connection ~ 3500 2700
 $Comp
@@
 	5200 1650 5200 1750
 Wire Wire Line
-	5200 2250 5200 2400
-Wire Wire Line
-	5200 2400 5200 2550
+	5200 2250 5200 2550
 Wire Wire Line
 	4600 2550 4700 2550
@@
 	5200 2400 3450 2400
 Connection ~ 5200 2400
-$Comp
-L POT RV1
-U 1 1 53441167
-P 2350 4350
-F 0 "RV1" H 2350 4250 50  0000 C CNN
-F 1 "POT" H 2350 4350 50  0000 C CNN
-F 2 "" H 2350 4350 60  0000 C CNN
-F 3 "" H 2350 4350 60  0000 C CNN
-	1    2350 4350
-	1    0    0    -1
-$EndComp
-$Comp
-L VCC #PWR024
-U 1 1 53441179
-P 2000 4350
-F 0 "#PWR024" H 2000 4450 30  0001 C CNN
-F 1 "VCC" H 2000 4450 30  0000 C CNN
-F 2 "" H 2000 4350 60  0000 C CNN
-F 3 "" H 2000 4350 60  0000 C CNN
-	1    2000 4350
-	0    -1   -1   0
-$EndComp
-$Comp
-L GND #PWR025
-U 1 1 53441184
-P 2700 4350
-F 0 "#PWR025" H 2700 4350 30  0001 C CNN
-F 1 "GND" H 2700 4280 30  0001 C CNN
-F 2 "" H 2700 4350 60  0000 C CNN
-F 3 "" H 2700 4350 60  0000 C CNN
-	1    2700 4350
-	0    -1   -1   0
-$EndComp
-Wire Wire Line
-	2000 4350 2100 4350
-Wire Wire Line
-	2600 4350 2700 4350
-Text GLabel 2350 4100 0    60   Output ~ 0
-BRIGHTNESS
-Wire Wire Line
-	2350 4100 2350 4200
-Text GLabel 3550 2300 2    60   Input ~ 0
-BRIGHTNESS
-Wire Wire Line
-	3450 2300 3550 2300
-$Comp
-L JUMPER3 JP1
-U 1 1 534413EB
-P 3900 3300
-F 0 "JP1" H 3950 3200 40  0000 L CNN
-F 1 "AUTOBRGT" H 3900 3400 40  0000 C CNN
-F 2 "" H 3900 3300 60  0000 C CNN
-F 3 "" H 3900 3300 60  0000 C CNN
-	1    3900 3300
-	1    0    0    -1
-$EndComp
-$Comp
-L GND #PWR026
-U 1 1 534413FD
-P 4250 3300
-F 0 "#PWR026" H 4250 3300 30  0001 C CNN
-F 1 "GND" H 4250 3230 30  0001 C CNN
-F 2 "" H 4250 3300 60  0000 C CNN
-F 3 "" H 4250 3300 60  0000 C CNN
-	1    4250 3300
-	0    -1   -1   0
-$EndComp
-Wire Wire Line
-	3450 3350 3650 3350
-Wire Wire Line
-	3650 3300 3650 3350
-Wire Wire Line
-	3650 3350 3650 3400
-Wire Wire Line
-	3650 3400 3900 3400
-Connection ~ 3650 3350
-Wire Wire Line
-	4150 3300 4250 3300
 $Comp
 L SW_PUSH SW1
@@
 $EndComp
 $Comp
-L GND #PWR027
+L GND #PWR025
 U 1 1 53441552
 P 5050 3250
-F 0 "#PWR027" H 5050 3250 30  0001 C CNN
+F 0 "#PWR025" H 5050 3250 30  0001 C CNN
 F 1 "GND" H 5050 3180 30  0001 C CNN
 F 2 "" H 5050 3250 60  0000 C CNN
@@
 $EndComp
 $Comp
-L GND #PWR028
+L GND #PWR026
 U 1 1 5344155D
 P 5850 3250
-F 0 "#PWR028" H 5850 3250 30  0001 C CNN
+F 0 "#PWR026" H 5850 3250 30  0001 C CNN
 F 1 "GND" H 5850 3180 30  0001 C CNN
 F 2 "" H 5850 3250 60  0000 C CNN
@@
 NoConn ~ 3450 3050
 $Comp
-L PWR_FLAG #FLG029
+L PWR_FLAG #FLG027
 U 1 1 53441864
 P 10550 1950
-F 0 "#FLG029" H 10550 2045 30  0001 C CNN
+F 0 "#FLG027" H 10550 2045 30  0001 C CNN
 F 1 "PWR_FLAG" H 10550 2130 30  0000 C CNN
 F 2 "" H 10550 1950 60  0000 C CNN
@@
 Connection ~ 10550 1950
 $Comp
-L PWR_FLAG #FLG030
+L PWR_FLAG #FLG028
 U 1 1 5344187A
 P 750 2100
-F 0 "#FLG030" H 750 2195 30  0001 C CNN
+F 0 "#FLG028" H 750 2195 30  0001 C CNN
 F 1 "PWR_FLAG" H 750 2280 30  0000 C CNN
 F 2 "" H 750 2100 60  0000 C CNN
@@
 	750  2100 850  2100
 Connection ~ 850  2100
-$Comp
-L CONN_6 P2
-U 1 1 53444226
-P 7400 4400
-F 0 "P2" V 7350 4400 60  0000 C CNN
-F 1 "FTDI" V 7450 4400 60  0000 C CNN
-F 2 "" H 7400 4400 60  0000 C CNN
-F 3 "" H 7400 4400 60  0000 C CNN
-	1    7400 4400
-	0    -1   1    0
-$EndComp
 Text GLabel 3800 2850 2    60   BiDi ~ 0
 FTDI3
 Wire Wire Line
 	3450 2850 3800 2850
-Text GLabel 7350 3900 1    60   BiDi ~ 0
-FTDI3
-Wire Wire Line
-	7350 4050 7350 3900
-Text GLabel 7250 3900 1    60   BiDi ~ 0
-FTDI2
-Wire Wire Line
-	7250 3900 7250 4050
 Text GLabel 3800 2950 2    60   BiDi ~ 0
 FTDI2
 Wire Wire Line
 	3800 2950 3450 2950
-$Comp
-L C C8
-U 1 1 534444CA
-P 6800 4050
-F 0 "C8" H 6800 4150 40  0000 L CNN
-F 1 "100nF" H 6806 3965 40  0000 L CNN
-F 2 "" H 6838 3900 30  0000 C CNN
-F 3 "" H 6800 4050 60  0000 C CNN
-	1    6800 4050
-	0    1    1    0
-$EndComp
-Wire Wire Line
-	7150 4050 7000 4050
-Wire Wire Line
-	6600 2800 6600 4050
 Connection ~ 5500 2800
 $Comp
-L GND #PWR031
-U 1 1 534445B7
-P 7650 3850
-F 0 "#PWR031" H 7650 3850 30  0001 C CNN
-F 1 "GND" H 7650 3780 30  0001 C CNN
-F 2 "" H 7650 3850 60  0000 C CNN
-F 3 "" H 7650 3850 60  0000 C CNN
-	1    7650 3850
-	-1   0    0    1
-$EndComp
-Wire Wire Line
-	7650 3850 7650 4050
-$Comp
-L VCC #PWR032
-U 1 1 53444635
-P 7450 3850
-F 0 "#PWR032" H 7450 3950 30  0001 C CNN
-F 1 "VCC" H 7450 3950 30  0000 C CNN
-F 2 "" H 7450 3850 60  0000 C CNN
-F 3 "" H 7450 3850 60  0000 C CNN
-	1    7450 3850
-	1    0    0    -1
-$EndComp
-Wire Wire Line
-	7450 3850 7450 4050
-NoConn ~ 7550 4050
+L DS1307 U1
+U 1 1 53435651
+P 8500 2500
+F 0 "U1" H 8600 1300 60  0000 C CNN
+F 1 "DS1307" H 8500 2550 60  0000 C CNN
+F 2 "" H 8500 2500 60  0000 C CNN
+F 3 "" H 8500 2500 60  0000 C CNN
+	1    8500 2500
+	1    0    0    -1
+$EndComp
+NoConn ~ 3450 3350
+NoConn ~ 3450 2300
 $EndSCHEMATC

Commit message: dammit
Connections:
- net labels removed: FTDI2, FTDI3
- wire segments 82 -> 80
- no-connect marks 13 -> 14
Changed lines of the file:
@@
 LIBS:ds1307timer
 LIBS:open-project
+LIBS:neoclock-cache
 EELAYER 24 0
 EELAYER END
@@
 	750  2100 850  2100
 Connection ~ 850  2100
-Text GLabel 3800 2850 2    60   BiDi ~ 0
-FTDI3
-Wire Wire Line
-	3450 2850 3800 2850
-Text GLabel 3800 2950 2    60   BiDi ~ 0
-FTDI2
-Wire Wire Line
-	3800 2950 3450 2950
 Connection ~ 5500 2800
 $Comp
@@
 NoConn ~ 3450 3350
 NoConn ~ 3450 2300
+NoConn ~ 3450 2850
 $EndSCHEMATC

Commit message: updated to the new smaller, attiny84 based board
Parts:
- removed C2: 100nF, symbol C
- removed IC1: ATMEGA328P-A, TQFP32, symbol ATMEGA328P-A
- added F1: FUSE, symbol FUSE
- added IC1: ATTINY84-S, SO14, symbol ATTINY84-S
Connections:
- net labels added: HOUR, MINUTE, MISO, MOSI, NEODATA, PHOTOR, RESET, SCK
- wire segments 80 -> 71
- no-connect marks 14 -> 4
Other:
- moved on the sheet: BT1, C1, C3, C4, C5, C6, C7, K1, P1, R2, R3, U1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
