File: kicad/neoclock.sch (KiCad schematic (older format))
At the start: 27 parts, among them CON1 2.1mm 5V, IC1 ATMEGA328P-A, K1 NEOPIXEL, P1 ICSP, P2 FTDI, SW1 HOUR, SW2 MINUTE, U1 DS1307, X1 16Mhz, X2 32.768kHz

Commit message: new board has lots of changes
Parts:
- removed P2: FTDI, Pin_Headers:Pin_Header_Straight_1x06, symbol CONN_3X2
- added C9: 100nF, Capacitors_SMD:c_0805, symbol C
- added P2: FTDI, symbol CONN_6
- C4: footprint Capacitors_SMD:c_elec_4x4.5 -> Capacitors_Tantalum_SMD:TantalC_SizeA_EIA-3216_Wave
- PHOTOR1: footprint synicpretty:PHOTORESISTOR -> synic:jst-2-pth-ra
- R2: footprint Resistors_SMD:Resistor_SMD0805_ReflowWave -> (none)
Connections:
- net labels added: RXD, TXD
- wire segments 97 -> 102
- no-connect marks 12 -> 11
Changed lines of the file:
@@
 Wire Wire Line
 	7150 2250 7350 2250
-$Comp
-L R R2
-U 1 1 53435901
-P 3750 2700
-F 0 "R2" V 3830 2700 40  0000 C CNN
-F 1 "10k" V 3757 2701 40  0000 C CNN
-F 2 "Resistors_SMD:Resistor_SMD0805_ReflowWave" V 3680 2700 30  0001 C CNN
-F 3 "" H 3750 2700 30  0000 C CNN
-	1    3750 2700
-	0    1    1    0
-$EndComp
-Wire Wire Line
-	3450 2700 3500 2700
-$Comp
-L VCC #PWR013
-U 1 1 5343593A
-P 4100 2700
-F 0 "#PWR013" H 4100 2800 30  0001 C CNN
-F 1 "VCC" H 4100 2800 30  0000 C CNN
-F 2 "" H 4100 2700 60  0000 C CNN
-F 3 "" H 4100 2700 60  0000 C CNN
-	1    4100 2700
-	0    1    1    0
-$EndComp
-Wire Wire Line
-	4000 2700 4100 2700
+Wire Wire Line
+	3450 2700 5500 2700
 $Comp
 L BARREL_JACK CON1
@@
 F 0 "C4" H 4650 1050 50  0000 L CNN
 F 1 "10uF" H 4650 850 50  0000 L CNN
-F 2 "Capacitors_SMD:c_elec_4x4.5" H 4600 950 60  0001 C CNN
+F 2 "Capacitors_Tantalum_SMD:TantalC_SizeA_EIA-3216_Wave" H 4600 950 60  0001 C CNN
 F 3 "" H 4600 950 60  0000 C CNN
 	1    4600 950
@@
 Connection ~ 4250 1150
 $Comp
-L GND #PWR014
+L GND #PWR013
 U 1 1 5343FBB9
 P 4950 1150
-F 0 "#PWR014" H 4950 1150 30  0001 C CNN
+F 0 "#PWR013" H 4950 1150 30  0001 C CNN
 F 1 "GND" H 4950 1080 30  0001 C CNN
 F 2 "" H 4950 1150 60  0000 C CNN
@@
 $EndComp
 $Comp
-L VCC #PWR015
+L VCC #PWR014
 U 1 1 5343FBC4
 P 4950 750
-F 0 "#PWR015" H 4950 850 30  0001 C CNN
+F 0 "#PWR014" H 4950 850 30  0001 C CNN
 F 1 "VCC" H 4950 850 30  0000 C CNN
 F 2 "" H 4950 750 60  0000 C CNN
@@
 	3700 1650 3450 1650
 $Comp
-L VCC #PWR016
+L VCC #PWR015
 U 1 1 5343FD7A
 P 6650 1150
-F 0 "#PWR016" H 6650 1250 30  0001 C CNN
+F 0 "#PWR015" H 6650 1250 30  0001 C CNN
 F 1 "VCC" H 6650 1250 30  0000 C CNN
 F 2 "" H 6650 1150 60  0000 C CNN
@@
 Wire Wire Line
 	5750 1350 5500 1350
-Wire Wire Line
-	5500 1350 5500 2800
-Wire Wire Line
-	5500 2800 3500 2800
-Wire Wire Line
-	3500 2800 3500 2700
-Connection ~ 3500 2700
-$Comp
-L GND #PWR017
+$Comp
+L GND #PWR016
 U 1 1 5343FEAD
 P 6600 1350
-F 0 "#PWR017" H 6600 1350 30  0001 C CNN
+F 0 "#PWR016" H 6600 1350 30  0001 C CNN
 F 1 "GND" H 6600 1280 30  0001 C CNN
 F 2 "" H 6600 1350 60  0000 C CNN
@@
 NoConn ~ 3450 1350
 NoConn ~ 3450 1250
-NoConn ~ 3450 3550
 $Comp
 L PHOTOR PHOTOR1
@@
 F 0 "PHOTOR1" V 5280 2000 50  0000 C CNN
 F 1 "PHOTOR" V 5200 2000 50  0000 C CNN
-F 2 "synicpretty:PHOTORESISTOR" H 5200 2000 60  0001 C CNN
+F 2 "synic:jst-2-pth-ra" H 5200 2000 60  0001 C CNN
 F 3 "" H 5200 2000 60  0000 C CNN
 	1    5200 2000
@@
 $EndComp
 $Comp
-L VCC #PWR018
+L VCC #PWR017
 U 1 1 53441003
 P 5200 1650
-F 0 "#PWR018" H 5200 1750 30  0001 C CNN
+F 0 "#PWR017" H 5200 1750 30  0001 C CNN
 F 1 "VCC" H 5200 1750 30  0000 C CNN
 F 2 "" H 5200 1650 60  0000 C CNN
@@
 $EndComp
 $Comp
-L GND #PWR019
+L GND #PWR018
 U 1 1 5344100E
 P 4600 2550
-F 0 "#PWR019" H 4600 2550 30  0001 C CNN
+F 0 "#PWR018" H 4600 2550 30  0001 C CNN
 F 1 "GND" H 4600 2480 30  0001 C CNN
 F 2 "" H 4600 2550 60  0000 C CNN
@@
 $EndComp
 $Comp
-L GND #PWR020
+L GND #PWR019
 U 1 1 53441552
 P 5050 3250
-F 0 "#PWR020" H 5050 3250 30  0001 C CNN
+F 0 "#PWR019" H 5050 3250 30  0001 C CNN
 F 1 "GND" H 5050 3180 30  0001 C CNN
 F 2 "" H 5050 3250 60  0000 C CNN
@@
 $EndComp
 $Comp
-L GND #PWR021
+L GND #PWR020
 U 1 1 5344155D
 P 5850 3250
-F 0 "#PWR021" H 5850 3250 30  0001 C CNN
+F 0 "#PWR020" H 5850 3250 30  0001 C CNN
 F 1 "GND" H 5850 3180 30  0001 C CNN
 F 2 "" H 5850 3250 60  0000 C CNN
@@
 NoConn ~ 3450 3050
 $Comp
-L PWR_FLAG #FLG022
+L PWR_FLAG #FLG021
 U 1 1 53441864
 P 10550 1950
-F 0 "#FLG022" H 10550 2045 30  0001 C CNN
+F 0 "#FLG021" H 10550 2045 30  0001 C CNN
 F 1 "PWR_FLAG" H 10550 2130 30  0000 C CNN
 F 2 "" H 10550 1950 60  0000 C CNN
@@
 Connection ~ 10550 1950
 $Comp
-L PWR_FLAG #FLG023
+L PWR_FLAG #FLG022
 U 1 1 5344187A
 P 750 2100
-F 0 "#FLG023" H 750 2195 30  0001 C CNN
+F 0 "#FLG022" H 750 2195 30  0001 C CNN
 F 1 "PWR_FLAG" H 750 2280 30  0000 C CNN
 F 2 "" H 750 2100 60  0000 C CNN
@@
 	1    0    0    -1
 $EndComp
-NoConn ~ 3450 3350
 NoConn ~ 3450 2300
 $Comp
@@
 	4200 750  4950 750
 $Comp
-L VCC #PWR024
+L VCC #PWR023
 U 1 1 5343FC65
 P 6350 3750
-F 0 "#PWR024" H 6350 3850 30  0001 C CNN
+F 0 "#PWR023" H 6350 3850 30  0001 C CNN
 F 1 "VCC" H 6350 3850 30  0000 C CNN
 F 2 "" H 6350 3750 60  0000 C CNN
@@
 $EndComp
 $Comp
-L GND #PWR025
+L GND #PWR024
 U 1 1 53D3CCBD
 P 6400 3350
-F 0 "#PWR025" H 6400 3350 30  0001 C CNN
+F 0 "#PWR024" H 6400 3350 30  0001 C CNN
 F 1 "GND" H 6400 3280 30  0001 C CNN
 F 2 "" H 6400 3350 60  0000 C CNN
@@
 $EndComp
 Wire Wire Line
-	5700 2850 3450 2850
-Wire Wire Line
 	5700 2750 5700 2850
-Wire Wire Line
-	5950 2950 3450 2950
 Wire Wire Line
 	5950 2750 5950 2950
@@
 $EndComp
 $Comp
-L GND #PWR026
+L GND #PWR025
 U 1 1 53D3E10F
 P 6300 1750
-F 0 "#PWR026" H 6300 1750 30  0001 C CNN
+F 0 "#PWR025" H 6300 1750 30  0001 C CNN
 F 1 "GND" H 6300 1680 30  0001 C CNN
 F 2 "" H 6300 1750 60  0000 C CNN
@@
 	5700 1750 6300 1750
 Connection ~ 5950 1750
-$Comp
-L CONN_3X2 P2
-U 1 1 53D3E5F5
-P 3900 4800
-F 0 "P2" H 3900 5050 50  0000 C CNN
-F 1 "FTDI" V 3900 4850 40  0000 C CNN
-F 2 "Pin_Headers:Pin_Header_Straight_1x06" H 3900 4800 60  0000 C CNN
-F 3 "" H 3900 4800 60  0000 C CNN
-	1    3900 4800
-	1    0    0    -1
-$EndComp
-Text GLabel 3400 4650 0    60   BiDi ~ 0
-MISO
-Text GLabel 3400 4750 0    60   BiDi ~ 0
-SCK
-Text GLabel 3400 4850 0    60   BiDi ~ 0
-RST
-Text GLabel 4400 4750 2    60   BiDi ~ 0
-MOSI
-$Comp
-L GND #PWR027
-U 1 1 53D3EA54
-P 4400 4850
-F 0 "#PWR027" H 4400 4850 30  0001 C CNN
-F 1 "GND" H 4400 4780 30  0001 C CNN
-F 2 "" H 4400 4850 60  0000 C CNN
-F 3 "" H 4400 4850 60  0000 C CNN
-	1    4400 4850
-	0    -1   -1   0
-$EndComp
-$Comp
-L VCC #PWR028
-U 1 1 53D3EA9F
-P 4400 4650
-F 0 "#PWR028" H 4400 4750 30  0001 C CNN
-F 1 "VCC" H 4400 4750 30  0000 C CNN
-F 2 "" H 4400 4650 60  0000 C CNN
-F 3 "" H 4400 4650 60  0000 C CNN
-	1    4400 4650
-	0    1    1    0
-$EndComp
-Wire Wire Line
-	3400 4650 3500 4650
-Wire Wire Line
-	3400 4750 3500 4750
-Wire Wire Line
-	3400 4850 3500 4850
-Wire Wire Line
-	4300 4650 4400 4650
-Wire Wire Line
-	4300 4750 4400 4750
-Wire Wire Line
-	4300 4850 4400 4850
 Text GLabel 5600 1600 2    60   BiDi ~ 0
 RST
@@
 	4800 1450 4800 1400
 Connection ~ 4800 1400
+Connection ~ 5500 2700
+Wire Wire Line
+	5500 1350 5500 2700
+Wire Wire Line
+	5950 2950 3850 2950
+Wire Wire Line
+	3850 2950 3850 3350
+Wire Wire Line
+	3850 3350 3450 3350
+Wire Wire Line
+	5700 2850 3800 2850
+Wire Wire Line
+	3800 2850 3800 3550
+Wire Wire Line
+	3800 3550 3450 3550
+$Comp
+L CONN_6 P2
+U 1 1 53D91495
+P 3900 4550
+F 0 "P2" V 3850 4550 60  0000 C CNN
+F 1 "FTDI" V 3950 4550 60  0000 C CNN
+F 2 "" H 3900 4550 60  0000 C CNN
+F 3 "" H 3900 4550 60  0000 C CNN
+	1    3900 4550
+	0    -1   1    0
+$EndComp
+$Comp
+L C C9
+U 1 1 53D91643
+P 3300 4200
+F 0 "C9" H 3300 4300 40  0000 L CNN
+F 1 "100nF" H 3306 4115 40  0000 L CNN
+F 2 "Capacitors_SMD:c_0805" H 3338 4050 30  0001 C CNN
+F 3 "" H 3300 4200 60  0000 C CNN
+	1    3300 4200
+	0    -1   -1   0
+$EndComp
+Text GLabel 3000 4200 0    60   BiDi ~ 0
+RST
+Wire Wire Line
+	3000 4200 3100 4200
+Wire Wire Line
+	3500 4200 3650 4200
+$Comp
+L R R2
+U 1 1 53D91853
+P 6300 1500
+F 0 "R2" V 6380 1500 40  0000 C CNN
+F 1 "10k" V 6307 1501 40  0000 C CNN
+F 2 "" V 6230 1500 30  0000 C CNN
+F 3 "" H 6300 1500 30  0000 C CNN
+	1    6300 1500
+	0    1    1    0
+$EndComp
+Wire Wire Line
+	5500 1500 6050 1500
+Connection ~ 5500 1500
+$Comp
+L VCC #PWR026
+U 1 1 53D919CE
+P 6600 1500
+F 0 "#PWR026" H 6600 1600 30  0001 C CNN
+F 1 "VCC" H 6600 1600 30  0000 C CNN
+F 2 "" H 6600 1500 60  0000 C CNN
+F 3 "" H 6600 1500 60  0000 C CNN
+	1    6600 1500
+	0    1    1    0
+$EndComp
+Wire Wire Line
+	6550 1500 6600 1500
+Text GLabel 3550 2850 2    60   BiDi ~ 0
+RXD
+Text GLabel 3550 2950 2    60   BiDi ~ 0
+TXD
+Wire Wire Line
+	3450 2850 3550 2850
+Wire Wire Line
+	3450 2950 3550 2950
+Text GLabel 3750 4150 1    60   BiDi ~ 0
+TXD
+Text GLabel 3850 4150 1    60   BiDi ~ 0
+RXD
+Wire Wire Line
+	3750 4150 3750 4200
+Wire Wire Line
+	3850 4150 3850 4200
+$Comp
+L VCC #PWR027
+U 1 1 53D920F9
+P 3950 4150
+F 0 "#PWR027" H 3950 4250 30  0001 C CNN
+F 1 "VCC" H 3950 4250 30  0000 C CNN
+F 2 "" H 3950 4150 60  0000 C CNN
+F 3 "" H 3950 4150 60  0000 C CNN
+	1    3950 4150
+	1    0    0    -1
+$EndComp
+Wire Wire Line
+	3950 4150 3950 4200
+NoConn ~ 4050 4200
+$Comp
+L GND #PWR028
+U 1 1 53D921BE
+P 4150 4150
+F 0 "#PWR028" H 4150 4150 30  0001 C CNN
+F 1 "GND" H 4150 4080 30  0001 C CNN
+F 2 "" H 4150 4150 60  0000 C CNN
+F 3 "" H 4150 4150 60  0000 C CNN
+	1    4150 4150
+	-1   0    0    1
+$EndComp
+Wire Wire Line
+	4150 4200 4150 4150
 $EndSCHEMATC

Commit message: lots of code updates
Parts:
- CON1: footprint synic:BARREL_JACK_SMD -> synicpretty:BARREL_JACK_SMD
- P2: footprint (none) -> Pin_Headers:Pin_Header_Straight_1x06
- R2: footprint (none) -> Resistors_SMD:Resistor_SMD0805_ReflowWave
Changed lines of the file:
@@
 F 0 "CON1" H 3400 1100 60  0000 C CNN
 F 1 "2.1mm 5V" H 3400 650 60  0000 C CNN
-F 2 "synic:BARREL_JACK_SMD" H 3400 850 60  0001 C CNN
+F 2 "synicpretty:BARREL_JACK_SMD" H 3400 850 60  0001 C CNN
 F 3 "" H 3400 850 60  0000 C CNN
 	1    3400 850
@@
 F 0 "P2" V 3850 4550 60  0000 C CNN
 F 1 "FTDI" V 3950 4550 60  0000 C CNN
-F 2 "" H 3900 4550 60  0000 C CNN
+F 2 "Pin_Headers:Pin_Header_Straight_1x06" H 3900 4550 60  0001 C CNN
 F 3 "" H 3900 4550 60  0000 C CNN
 	1    3900 4550
@@
 F 0 "R2" V 6380 1500 40  0000 C CNN
 F 1 "10k" V 6307 1501 40  0000 C CNN
-F 2 "" V 6230 1500 30  0000 C CNN
+F 2 "Resistors_SMD:Resistor_SMD0805_ReflowWave" V 6230 1500 30  0001 C CNN
 F 3 "" H 6300 1500 30  0000 C CNN
 	1    6300 1500

Commit message: sweet
Parts:
- removed BT1: BATTERY, synicpretty:BK-755_12mm_coincell, symbol BATTERY
- removed C1, C2, C7, C9: 100nF, Capacitors_SMD:c_0805, symbol C
- removed C3, C8: 100uF, Capacitors_SMD:c_elec_5x5.3, symbol CP1
- removed C4: 10uF, Capacitors_Tantalum_SMD:TantalC_SizeA_EIA-3216_Wave, symbol CP1
- removed C5, C6: 22pF, Capacitors_SMD:c_0805, symbol C
- removed CON1: 2.1mm 5V, synicpretty:BARREL_JACK_SMD, symbol BARREL_JACK
- removed D1: ERROR, LEDs:LED-0805, symbol LED
- removed D2: PWR, LEDs:LED-0805, symbol LED
- removed F1: FUSE, synic:1206_polyfuse, symbol FUSE
- removed IC1: ATMEGA328P-A, SMD_Packages:TQFP32, symbol ATMEGA328P-A
- removed K1: NEOPIXEL, synic:jst-3-pth-ra, symbol CONN_3
- removed P1: ICSP, Pin_Headers:Pin_Header_Straight_2x03, symbol CONN_3X2
- removed P2: FTDI, Pin_Headers:Pin_Header_Straight_1x06, symbol CONN_6
- removed PHOTOR1: PHOTOR, synic:jst-2-pth-ra, symbol PHOTOR
- removed R1, R4: 330, Resistors_SMD:Resistor_SMD0805_ReflowWave, symbol R
- removed R2, R3: 10k, Resistors_SMD:Resistor_SMD0805_ReflowWave, symbol R
- removed SW1: HOUR, synic:KMR2_MICROMINIATURE_BUTTON, symbol SW_PUSH
- removed SW2: MINUTE, synic:KMR2_MICROMINIATURE_BUTTON, symbol SW_PUSH
- removed U1: DS1307, SOIC_Packages:SOIC-8_N, symbol DS1307
- removed X1: 16Mhz, synic:2_SMD_CRYSTAL_5.0x3.20, symbol CRYSTAL
- removed X2: 32.768kHz, synic:2_SMD_CRYSTAL_3.2x1.5, symbol CRYSTAL
- added BT?: 3v, symbol BATTERY
- added C?: 10nF, symbol C
- added C?: 1uF, symbol C
- added C? (x3): 100nF, symbol C
- added C?: 4.7uF, symbol C
- added C? (x2): 18pF, symbol C
- added C? (x2): 10uF, symbol CP1
- added C?: 100uF, symbol CP1
- added CON?: 1.2mm 5v, symbol BARREL_JACK
- added K?: NEO, symbol CONN_3
- added P?: TC2030-CTX, symbol TC2030-CTX
- added R? (x2): 10k, symbol R
- added U?: stm32f303x, symbol stm32f303x
- added U?: 7805, symbol 7805
- added X?: 32.768KHz, symbol CRYSTAL
- added X?: 8MHz, symbol CRYSTAL
Connections:
- net labels added: NRST, SWCLK, SWDIO, VDD
- net labels removed: I2CSCL, I2CSDA, MISO, MOSI, RST, RXD, SCK, TXD, VCC
- wire segments 102 -> 50
- no-connect marks 11 -> 1

Commit message: stuff
Parts:
- C?: value 100uF -> 470uF
- U?: value 7805 -> 3.3V REG
Connections:
- wire segments 50 -> 48
Other:
- moved on the sheet: C?
Changed lines of the file:
@@
 P 7400 950
 F 0 "U?" H 7550 754 60  0000 C CNN
-F 1 "7805" H 7400 1150 60  0000 C CNN
+F 1 "3.3V REG" H 7400 1150 60  0000 C CNN
 F 2 "" H 7400 950 60  0000 C CNN
 F 3 "" H 7400 950 60  0000 C CNN
@@
 L CP1 C?
 U 1 1 5420AA5E
-P 5550 1400
-F 0 "C?" H 5600 1500 50  0000 L CNN
-F 1 "100uF" H 5600 1300 50  0000 L CNN
-F 2 "" H 5550 1400 60  0000 C CNN
-F 3 "" H 5550 1400 60  0000 C CNN
-	1    5550 1400
+P 5400 850
+F 0 "C?" H 5450 950 50  0000 L CNN
+F 1 "470uF" H 5450 750 50  0000 L CNN
+F 2 "" H 5400 850 60  0000 C CNN
+F 3 "" H 5400 850 60  0000 C CNN
+	1    5400 850
 	1    0    0    -1
 $EndComp
@@
 Connection ~ 6750 900
 Wire Wire Line
-	6400 900  6400 650
+	6400 650  6400 900
 Wire Wire Line
-	6400 650  5550 650
-Wire Wire Line
-	5550 650  5550 1200
+	5050 650  6400 650
 Wire Wire Line
 	6400 1000 6400 1300
@@
 $EndComp
 Wire Wire Line
-	5550 1200 5050 1200
-Wire Wire Line
-	5050 1200 5050 1850
+	5050 650  5050 1850
 Wire Wire Line
 	5050 1850 5200 1850
-Wire Wire Line
-	5550 1600 5400 1600
 $Comp
 L GND #PWR?
 U 1 1 5420B529
-P 5400 1600
-F 0 "#PWR?" H 5400 1600 30  0001 C CNN
-F 1 "GND" H 5400 1530 30  0001 C CNN
-F 2 "" H 5400 1600 60  0000 C CNN
-F 3 "" H 5400 1600 60  0000 C CNN
-	1    5400 1600
-	0    1    1    0
+P 5400 1200
+F 0 "#PWR?" H 5400 1200 30  0001 C CNN
+F 1 "GND" H 5400 1130 30  0001 C CNN
+F 2 "" H 5400 1200 60  0000 C CNN
+F 3 "" H 5400 1200 60  0000 C CNN
+	1    5400 1200
+	1    0    0    -1
 $EndComp
 $Comp
@@
 	0    1    1    0
 $EndComp
+Wire Wire Line
+	5400 1050 5400 1200
 $EndSCHEMATC

Commit message: schematic is mostly done
Parts:
- removed U?: stm32f303x, symbol stm32f303x
- added P2: PHOTOR, symbol CONN_2
- added R3: 10k, symbol R
- added SW1: HOUR, symbol SW_PUSH
- added SW2: MINUTE, symbol SW_PUSH
- added U1: stm32f303x, symbol stm32f303x
- gave numbers to parts that had none: 20
Connections:
- net labels added: VCC5V
- wire segments 48 -> 57
- no-connect marks 1 -> 28
Other:
- moved on the sheet: C10, C11, C9, CON1

Commit message: started to get somewhere here
Parts:
- removed C11: 10uF, symbol CP1
- removed C4: 18pF, symbol C
- removed U2: 3.3V REG, symbol 7805
- removed X2: 8MHz, symbol CRYSTAL
- added F1: FUSE, synic:1206_polyfuse, symbol FUSE
- added R4: 10k, Resistors_SMD:R_0603, symbol R
- added SW3: HOUR, synic:KMR2_MICROMINIATURE_BUTTON, symbol SW_PUSH
- added SW4: MINUTE, synic:KMR2_MICROMINIATURE_BUTTON, symbol SW_PUSH
- added U2: TLV702xx, SMD_Packages:SOT-23-5, symbol TLV702xx
- BT1: footprint (none) -> synicpretty:BK-755_12mm_coincell
- C1, C2, C5, C6, C7, C8: footprint (none) -> Capacitors_SMD:C_0603
- C10: footprint (none) -> Capacitors_SMD:c_elec_4x4.5
- C3: value 18pF -> 1uF
- C9: value 470uF -> 100uF; footprint (none) -> Capacitors_SMD:c_elec_5x5.3
- CON1: footprint (none) -> synicpretty:BARREL_JACK_SMD
- K1: footprint (none) -> synic:jst-3-pth-ra
- P1: footprint (none) -> Tag-Connect:TC2030_SMALL
- P2, SW1, SW2: footprint (none) -> synic:jst-2-pth-ra
- R1, R2, R3: footprint (none) -> Resistors_SMD:R_0603
- U1: footprint (none) -> lqfp48:LQFP48
- X1: footprint (none) -> synic:2_SMD_CRYSTAL_3.2x1.5
Connections:
- wire segments 57 -> 52
- no-connect marks 28 -> 30
Other:
- moved on the sheet: CON1, K1

Commit message: board is done?
Parts:
- C1, C2: footprint Capacitors_SMD:C_0603 -> Capacitors_SMD:C_0805
- C3: footprint (none) -> Capacitors_SMD:C_0805
Changed lines of the file:
@@
 F 0 "C2" H 1100 2400 40  0000 L CNN
 F 1 "1uF" H 1106 2215 40  0000 L CNN
-F 2 "Capacitors_SMD:C_0603" H 1138 2150 30  0001 C CNN
+F 2 "Capacitors_SMD:C_0805" H 1138 2150 30  0001 C CNN
 F 3 "" H 1100 2300 60  0000 C CNN
 	1    1100 2300
@@
 F 0 "C1" H 1100 1550 40  0000 L CNN
 F 1 "4.7uF" H 1106 1365 40  0000 L CNN
-F 2 "Capacitors_SMD:C_0603" H 1138 1300 30  0001 C CNN
+F 2 "Capacitors_SMD:C_0805" H 1138 1300 30  0001 C CNN
 F 3 "" H 1100 1450 60  0000 C CNN
 	1    1100 1450
@@
 F 0 "C3" H 4650 7400 40  0000 L CNN
 F 1 "1uF" H 4656 7215 40  0000 L CNN
-F 2 "" H 4688 7150 30  0000 C CNN
+F 2 "Capacitors_SMD:C_0805" H 4688 7150 30  0001 C CNN
 F 3 "" H 4650 7300 60  0000 C CNN
 	1    4650 7300

Commit message: stuff
Connections:
- net labels added: VCC
- wire segments 52 -> 53
Other:
- moved on the sheet: K1
Changed lines of the file:
@@
 LIBS:Tag-Connect
 LIBS:neoclock-cache
-EELAYER 24 0
+EELAYER 25 0
 EELAYER END
 $Descr A4 11693 8268
@@
 L CONN_3 K1
 U 1 1 5420A63C
-P 5150 1950
-F 0 "K1" V 5100 1950 50  0000 C CNN
-F 1 "NEO" V 5200 1950 40  0000 C CNN
-F 2 "synic:jst-3-pth-ra" H 5150 1950 60  0001 C CNN
-F 3 "" H 5150 1950 60  0000 C CNN
-	1    5150 1950
+P 5550 2650
+F 0 "K1" V 5500 2650 50  0000 C CNN
+F 1 "NEO" V 5600 2650 40  0000 C CNN
+F 2 "synic:jst-3-pth-ra" H 5550 2650 60  0001 C CNN
+F 3 "" H 5550 2650 60  0000 C CNN
+	1    5550 2650
 	1    0    0    -1
 $EndComp
@@
 L GND #PWR010
 U 1 1 5420B549
-P 4800 1950
-F 0 "#PWR010" H 4800 1950 30  0001 C CNN
-F 1 "GND" H 4800 1880 30  0001 C CNN
-F 2 "" H 4800 1950 60  0000 C CNN
-F 3 "" H 4800 1950 60  0000 C CNN
-	1    4800 1950
+P 5200 2650
+F 0 "#PWR010" H 5200 2650 30  0001 C CNN
+F 1 "GND" H 5200 2580 30  0001 C CNN
+F 2 "" H 5200 2650 60  0000 C CNN
+F 3 "" H 5200 2650 60  0000 C CNN
+	1    5200 2650
 	0    1    1    0
 $EndComp
@@
 Connection ~ 1300 1650
 Connection ~ 1100 1650
-Wire Wire Line
-	1350 2500 1350 2750
-Connection ~ 1350 2500
 Connection ~ 1350 2650
 Wire Wire Line
@@
 Wire Wire Line
 	2600 4950 2650 4950
-Wire Wire Line
-	4150 2050 4800 2050
 Wire Wire Line
 	2100 7100 3650 7100
@@
 Connection ~ 4650 7500
 Wire Wire Line
-	4700 1850 4800 1850
+	5100 2550 5200 2550
 Wire Wire Line
 	2650 6700 2650 6850
@@
 Text GLabel 3200 6300 2    60   Output ~ 0
 VCC5V
-Text GLabel 4700 1850 0    60   Input ~ 0
+Text GLabel 5100 2550 0    60   Input ~ 0
 VCC5V
 Wire Wire Line
@@
 NoConn ~ 4150 2250
 NoConn ~ 4150 2550
-NoConn ~ 4150 2750
 NoConn ~ 4150 2850
 NoConn ~ 4150 2950
@@
 $EndComp
 Connection ~ 1100 1700
+Wire Wire Line
+	1350 2650 1350 2750
+Wire Wire Line
+	1350 2750 1200 2750
+$Comp
+L VCC #PWR?
+U 1 1 543089E2
+P 1200 2750
+F 0 "#PWR?" H 1200 2850 30  0001 C CNN
+F 1 "VCC" H 1200 2850 30  0000 C CNN
+F 2 "" H 1200 2750 60  0000 C CNN
+F 3 "" H 1200 2750 60  0000 C CNN
+	1    1200 2750
+	0    -1   -1   0
+$EndComp
+Wire Wire Line
+	4150 2750 5200 2750
+NoConn ~ 4150 2050
 $EndSCHEMATC
