File: kicad/neoclock.sch (KiCad schematic (older format))
At the start: 26 parts, among them CON1 1.2mm 5v, K1 NEO, P1 TC2030-CTX, P2 PHOTOR, SW1 HOUR, SW2 MINUTE, SW3 HOUR, SW4 MINUTE, U1 stm32f303x, U2 TLV702xx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

Commit message: wooters
Parts:
- removed SW3: HOUR, synic:KMR2_MICROMINIATURE_BUTTON, symbol SW_PUSH
- removed SW4: MINUTE, synic:KMR2_MICROMINIATURE_BUTTON, symbol SW_PUSH
- added C11, C4: 100nF, Capacitors_SMD:C_0805, symbol C
- added D1: RED, LEDs:LED-0805, symbol LED
- added D2: GREEN, LEDs:LED-0805, symbol LED
- added R5, R6: 330, Resistors_SMD:R_0805, symbol R
- added U3: TXS0101, SMD_Packages:SOT-23-6, symbol TXS0101
- added U4: NEO, synicpretty:TESTPOINT, symbol TESTPOINT
- added U5: GND, synicpretty:TESTPOINT, symbol TESTPOINT
- added U6: VCC5V, synicpretty:TESTPOINT, symbol TESTPOINT
- C5, C6, C7, C8: footprint Capacitors_SMD:C_0603 -> Capacitors_SMD:C_0805
- R1, R2, R3, R4: footprint Resistors_SMD:R_0603 -> Resistors_SMD:R_0805
- SW1, SW2: footprint synic:jst-2-pth-ra -> synic:KMR2_MICROMINIATURE_BUTTON
Connections:
- net labels removed: VCC
- wire segments 53 -> 71
- no-connect marks 30 -> 28
Other:
- moved on the sheet: K1

Commit message: bleh
Connections:
- wire segments 71 -> 72
Changed lines of the file:
@@
 	4150 2050 4700 2050
-Wire Wire Line
-	5500 1950 6100 1950
 Wire Wire Line
 	6100 1850 6100 2200
 Connection ~ 6100 1850
-Connection ~ 6100 1950
 $Comp
 L GND #PWR016
@@
 	5950 1250 5950 750
 Wire Wire Line
-	4450 1550 4700 1550
+	4450 1550 5600 1550
 Wire Wire Line
 	4450 1950 4700 1950
@@
 	1450 6400 1450 7100
 Connection ~ 1450 7100
+Wire Wire Line
+	5500 1950 5600 1950
+Wire Wire Line
+	5600 1950 5600 1550
+Connection ~ 4700 1550
 $EndSCHEMATC

Commit message: fixed the board
Parts:
- removed C11, C4: 100nF, Capacitors_SMD:C_0805, symbol C
- removed U3: TXS0101, SMD_Packages:SOT-23-6, symbol TXS0101
Connections:
- wire segments 72 -> 66
Other:
- moved on the sheet: K1
Changed lines of the file:
@@
 LIBS:Tag-Connect
 LIBS:neoclock-cache
-EELAYER 24 0
+EELAYER 25 0
 EELAYER END
 $Descr A4 11693 8268
@@
 L CONN_3 K1
 U 1 1 5420A63C
-P 6950 1950
-F 0 "K1" V 6900 1950 50  0000 C CNN
-F 1 "NEO" V 7000 1950 40  0000 C CNN
-F 2 "synic:jst-3-pth-ra" H 6950 1950 60  0001 C CNN
-F 3 "" H 6950 1950 60  0000 C CNN
-	1    6950 1950
+P 6000 2100
+F 0 "K1" V 5950 2100 50  0000 C CNN
+F 1 "NEO" V 6050 2100 40  0000 C CNN
+F 2 "synic:jst-3-pth-ra" H 6000 2100 60  0001 C CNN
+F 3 "" H 6000 2100 60  0000 C CNN
+	1    6000 2100
 	1    0    0    -1
 $EndComp
@@
 L GND #PWR010
 U 1 1 5420B549
-P 6600 1950
-F 0 "#PWR010" H 6600 1950 30  0001 C CNN
-F 1 "GND" H 6600 1880 30  0001 C CNN
-F 2 "" H 6600 1950 60  0000 C CNN
-F 3 "" H 6600 1950 60  0000 C CNN
-	1    6600 1950
+P 5600 2100
+F 0 "#PWR010" H 5600 2100 30  0001 C CNN
+F 1 "GND" H 5600 2030 30  0001 C CNN
+F 2 "" H 5600 2100 60  0000 C CNN
+F 3 "" H 5600 2100 60  0000 C CNN
+	1    5600 2100
 	0    1    1    0
 $EndComp
@@
 Connection ~ 1300 1650
 Connection ~ 1100 1650
-Connection ~ 1350 2650
 Wire Wire Line
 	1850 2650 1950 2650
@@
 Connection ~ 4650 7500
 Wire Wire Line
-	5500 1850 6600 1850
-Wire Wire Line
 	2650 6700 2650 6850
 Wire Wire Line
@@
 Connection ~ 2650 6300
 Text GLabel 3200 6300 2    60   Output ~ 0
-VCC5V
-Text GLabel 6100 2200 3    60   Input ~ 0
 VCC5V
 Wire Wire Line
@@
 NoConn ~ 4150 1450
 NoConn ~ 4150 1550
-NoConn ~ 4150 1650
 NoConn ~ 4150 1750
 NoConn ~ 4150 1850
@@
 L stm32f303x U1
 U 1 1 5420ED70
-P 3050 2850
-F 0 "U1" H 3050 4800 60  0000 C CNN
-F 1 "stm32f303x" H 3050 1450 60  0000 C CNN
-F 2 "lqfp48:LQFP48" H 3050 2850 60  0001 C CNN
-F 3 "" H 3050 2850 60  0000 C CNN
-	1    3050 2850
+P 3150 2300
+F 0 "U1" H 3150 4250 60  0000 C CNN
+F 1 "stm32f303x" H 3150 900 60  0000 C CNN
+F 2 "lqfp48:LQFP48" H 3150 2300 60  0001 C CNN
+F 3 "" H 3150 2300 60  0000 C CNN
+	1    3150 2300
 	1    0    0    -1
 $EndComp
@@
 Connection ~ 1100 1700
 Wire Wire Line
-	1350 2650 1350 2750
-Wire Wire Line
 	1350 2750 1200 2750
 $Comp
@@
 	5400 2850 5500 2850
 Connection ~ 5400 2850
-$Comp
-L TXS0101 U3
-U 1 1 5431C46F
-P 5100 1900
-F 0 "U3" H 5100 1600 60  0000 C CNN
-F 1 "TXS0101" H 5100 2100 60  0000 C CNN
-F 2 "SMD_Packages:SOT-23-6" H 5100 1900 60  0001 C CNN
-F 3 "" H 5100 1900 60  0000 C CNN
-	1    5100 1900
-	1    0    0    -1
-$EndComp
-Wire Wire Line
-	4150 2050 4700 2050
-Wire Wire Line
-	6100 1850 6100 2200
-Connection ~ 6100 1850
-$Comp
-L GND #PWR016
-U 1 1 5431CCFA
-P 4450 1950
-F 0 "#PWR016" H 4450 1950 30  0001 C CNN
-F 1 "GND" H 4450 1880 30  0001 C CNN
-F 2 "" H 4450 1950 60  0000 C CNN
-F 3 "" H 4450 1950 60  0000 C CNN
-	1    4450 1950
-	0    1    1    0
-$EndComp
-Wire Wire Line
-	4700 1550 4700 1850
-$Comp
-L C C4
-U 1 1 5431D491
-P 4550 1750
-F 0 "C4" H 4550 1850 40  0000 L CNN
-F 1 "100nF" H 4556 1665 40  0000 L CNN
-F 2 "Capacitors_SMD:C_0805" H 4588 1600 30  0001 C CNN
-F 3 "" H 4550 1750 60  0000 C CNN
-	1    4550 1750
-	1    0    0    -1
-$EndComp
-Connection ~ 4550 1550
-$Comp
-L C C11
-U 1 1 5431D76D
-P 6350 2050
-F 0 "C11" H 6350 2150 40  0000 L CNN
-F 1 "100nF" H 6356 1965 40  0000 L CNN
-F 2 "Capacitors_SMD:C_0805" H 6388 1900 30  0001 C CNN
-F 3 "" H 6350 2050 60  0000 C CNN
-	1    6350 2050
-	1    0    0    -1
-$EndComp
-Connection ~ 6350 1850
-$Comp
-L GND #PWR017
-U 1 1 5431D7F0
-P 6350 2300
-F 0 "#PWR017" H 6350 2300 30  0001 C CNN
-F 1 "GND" H 6350 2230 30  0001 C CNN
-F 2 "" H 6350 2300 60  0000 C CNN
-F 3 "" H 6350 2300 60  0000 C CNN
-	1    6350 2300
-	1    0    0    -1
-$EndComp
-Wire Wire Line
-	6350 2300 6350 2250
-Wire Wire Line
-	5500 2050 5500 2550
-Wire Wire Line
-	5500 2550 6600 2550
-Wire Wire Line
-	6600 2550 6600 2050
+Wire Wire Line
+	5100 2200 5650 2200
 $Comp
 L TESTPOINT U4
 U 1 1 5431DE36
-P 6100 3300
-F 0 "U4" H 6100 3200 60  0000 C CNN
-F 1 "NEO" H 6100 3500 60  0000 C CNN
-F 2 "synicpretty:TESTPOINT" H 6200 3300 60  0001 C CNN
-F 3 "" H 6200 3300 60  0000 C CNN
-	1    6100 3300
-	1    0    0    -1
-$EndComp
-Wire Wire Line
-	5800 3250 5800 2550
-Connection ~ 5800 2550
+P 5900 2950
+F 0 "U4" H 5900 2850 60  0000 C CNN
+F 1 "NEO" H 5900 3150 60  0000 C CNN
+F 2 "synicpretty:TESTPOINT" H 6000 2950 60  0001 C CNN
+F 3 "" H 6000 2950 60  0000 C CNN
+	1    5900 2950
+	1    0    0    -1
+$EndComp
+Wire Wire Line
+	5600 2900 5600 2200
+Connection ~ 5600 2200
 $Comp
 L TESTPOINT U5
 U 1 1 5431DF40
-P 6100 3700
-F 0 "U5" H 6100 3600 60  0000 C CNN
-F 1 "GND" H 6100 3900 60  0000 C CNN
-F 2 "synicpretty:TESTPOINT" H 6200 3700 60  0001 C CNN
-F 3 "" H 6200 3700 60  0000 C CNN
-	1    6100 3700
+P 5050 3700
+F 0 "U5" H 5050 3600 60  0000 C CNN
+F 1 "GND" H 5050 3900 60  0000 C CNN
+F 2 "synicpretty:TESTPOINT" H 5150 3700 60  0001 C CNN
+F 3 "" H 5150 3700 60  0000 C CNN
+	1    5050 3700
 	1    0    0    -1
 $EndComp
@@
 L GND #PWR018
 U 1 1 5431DFE3
-P 5700 3650
-F 0 "#PWR018" H 5700 3650 30  0001 C CNN
-F 1 "GND" H 5700 3580 30  0001 C CNN
-F 2 "" H 5700 3650 60  0000 C CNN
-F 3 "" H 5700 3650 60  0000 C CNN
-	1    5700 3650
-	0    1    1    0
-$EndComp
-Wire Wire Line
-	5700 3650 5800 3650
+P 4650 3650
+F 0 "#PWR018" H 4650 3650 30  0001 C CNN
+F 1 "GND" H 4650 3580 30  0001 C CNN
+F 2 "" H 4650 3650 60  0000 C CNN
+F 3 "" H 4650 3650 60  0000 C CNN
+	1    4650 3650
+	0    1    1    0
+$EndComp
+Wire Wire Line
+	4650 3650 4750 3650
 $Comp
 L TESTPOINT U6
@@
 Wire Wire Line
 	5950 1250 5950 750
-Wire Wire Line
-	4450 1550 5600 1550
-Wire Wire Line
-	4450 1950 4700 1950
-Connection ~ 4550 1950
-$Comp
-L VDD #PWR019
-U 1 1 5431F998
-P 4450 1550
-F 0 "#PWR019" H 4450 1650 30  0001 C CNN
-F 1 "VDD" H 4450 1660 30  0000 C CNN
-F 2 "" H 4450 1550 60  0000 C CNN
-F 3 "" H 4450 1550 60  0000 C CNN
-	1    4450 1550
-	0    -1   -1   0
-$EndComp
 $Comp
 L VDD #PWR020
@@
 	1450 6400 1450 7100
 Connection ~ 1450 7100
-Wire Wire Line
-	5500 1950 5600 1950
-Wire Wire Line
-	5600 1950 5600 1550
-Connection ~ 4700 1550
+NoConn ~ 4150 2050
+Wire Wire Line
+	4150 1650 5100 1650
+Wire Wire Line
+	5100 1650 5100 2200
+Wire Wire Line
+	1350 2650 900  2650
+Wire Wire Line
+	900  2650 900  2500
+Connection ~ 900  2500
+Wire Wire Line
+	5600 2100 5650 2100
+Text GLabel 5550 2000 0    60   Output ~ 0
+VCC5V
+Wire Wire Line
+	5650 2000 5550 2000
 $EndSCHEMATC

Commit message: updating
Parts:
- removed BT1: 3v, synicpretty:BK-755_12mm_coincell, symbol BATTERY
- removed K1: NEO, synic:jst-3-pth-ra, symbol CONN_3
- removed P2: PHOTOR, synic:jst-2-pth-ra, symbol CONN_2
- removed R3: 10k, Resistors_SMD:R_0805, symbol R
- removed X1: 32.768KHz, synic:2_SMD_CRYSTAL_3.2x1.5, symbol CRYSTAL
- added BT1: 3v, synicpretty:BK-755_12mm_coincell, symbol Battery
- added P2: CONN_01X03, synic:jst-3-pth-ra, symbol CONN_01X03
- added Y1: 32.768 KHz, synic:2_SMD_CRYSTAL_3.2x1.5, symbol Crystal_Small
- U2: footprint SMD_Packages:SOT-23-5 -> SOT23-5:SOT23-5
Connections:
- wire segments 66 -> 81
- no-connect marks 28 -> 29
Changed lines of the file:
@@
 LIBS:memory
 LIBS:xilinx
-LIBS:special
 LIBS:microcontrollers
 LIBS:dsp
@@
 $EndDescr
 $Comp
-L BATTERY BT1
-U 1 1 54207155
-P 1650 4800
-F 0 "BT1" H 1650 5000 50  0000 C CNN
-F 1 "3v" H 1650 4610 50  0000 C CNN
-F 2 "synicpretty:BK-755_12mm_coincell" H 1650 4800 60  0001 C CNN
-F 3 "" H 1650 4800 60  0000 C CNN
-	1    1650 4800
-	-1   0    0    1
-$EndComp
-$Comp
 L C C6
 U 1 1 542083CF
@@
 $EndComp
 $Comp
-L CRYSTAL X1
-U 1 1 5420907D
-P 1700 3300
-F 0 "X1" H 1700 3450 60  0000 C CNN
-F 1 "32.768KHz" H 1700 3150 60  0000 C CNN
-F 2 "synic:2_SMD_CRYSTAL_3.2x1.5" H 1700 3300 60  0001 C CNN
-F 3 "" H 1700 3300 60  0000 C CNN
-	1    1700 3300
-	0    1    1    0
-$EndComp
-$Comp
 L GND #PWR04
 U 1 1 5420967D
-P 1200 4800
-F 0 "#PWR04" H 1200 4800 30  0001 C CNN
-F 1 "GND" H 1200 4730 30  0001 C CNN
-F 2 "" H 1200 4800 60  0000 C CNN
-F 3 "" H 1200 4800 60  0000 C CNN
-	1    1200 4800
+P 1450 4800
+F 0 "#PWR04" H 1450 4800 30  0001 C CNN
+F 1 "GND" H 1450 4730 30  0001 C CNN
+F 2 "" H 1450 4800 60  0000 C CNN
+F 3 "" H 1450 4800 60  0000 C CNN
+	1    1450 4800
 	0    1    1    0
 $EndComp
@@
 $EndComp
 $Comp
-L CONN_3 K1
-U 1 1 5420A63C
-P 6000 2100
-F 0 "K1" V 5950 2100 50  0000 C CNN
-F 1 "NEO" V 6050 2100 40  0000 C CNN
-F 2 "synic:jst-3-pth-ra" H 6000 2100 60  0001 C CNN
-F 3 "" H 6000 2100 60  0000 C CNN
-	1    6000 2100
-	1    0    0    -1
-$EndComp
-$Comp
 L BARREL_JACK CON1
 U 1 1 5420A944
@@
 Connection ~ 1500 1650
 Wire Wire Line
-	1100 1650 1100 1750
+	1100 1600 1100 1750
 Connection ~ 1300 1250
 Connection ~ 1300 1650
 Connection ~ 1100 1650
 Wire Wire Line
-	1850 2650 1950 2650
-Wire Wire Line
-	1850 2750 1950 2750
-Wire Wire Line
-	1950 3000 1950 3100
-Wire Wire Line
-	1950 3600 1950 3500
+	1750 2650 1950 2650
+Wire Wire Line
+	1750 2750 1950 2750
 Wire Wire Line
 	1950 4450 1950 4800
@@
 Connection ~ 4650 7500
 Wire Wire Line
-	2650 6700 2650 6850
+	2650 6650 2650 6850
 Wire Wire Line
 	2350 6300 3200 6300
@@
 Text GLabel 3200 6300 2    60   Output ~ 0
 VCC5V
-Wire Wire Line
-	4150 1050 4900 1050
-$Comp
-L VDD #PWR011
-U 1 1 5420CFFF
-P 5200 1050
-F 0 "#PWR011" H 5200 1150 30  0001 C CNN
-F 1 "VDD" H 5200 1160 30  0000 C CNN
-F 2 "" H 5200 1050 60  0000 C CNN
-F 3 "" H 5200 1050 60  0000 C CNN
-	1    5200 1050
-	0    1    1    0
-$EndComp
-Wire Wire Line
-	5100 1050 5200 1050
-$Comp
-L GND #PWR012
-U 1 1 5420D0BD
-P 4150 900
-F 0 "#PWR012" H 4150 900 30  0001 C CNN
-F 1 "GND" H 4150 830 30  0001 C CNN
-F 2 "" H 4150 900 60  0000 C CNN
-F 3 "" H 4150 900 60  0000 C CNN
-	1    4150 900
-	0    1    1    0
-$EndComp
-$Comp
-L R R3
-U 1 1 5420D0CA
-P 4500 900
-F 0 "R3" V 4580 900 40  0000 C CNN
-F 1 "10k" V 4507 901 40  0000 C CNN
-F 2 "Resistors_SMD:R_0805" V 4430 900 30  0001 C CNN
-F 3 "" H 4500 900 30  0000 C CNN
-	1    4500 900
-	0    1    1    0
-$EndComp
-Wire Wire Line
-	4750 1050 4750 900
-Wire Wire Line
-	4250 900  4150 900
-$Comp
-L CONN_2 P2
-U 1 1 5420D3A0
-P 5000 700
-F 0 "P2" V 4950 700 40  0000 C CNN
-F 1 "PHOTOR" V 5050 700 40  0000 C CNN
-F 2 "synic:jst-2-pth-ra" H 5000 700 60  0001 C CNN
-F 3 "" H 5000 700 60  0000 C CNN
-	1    5000 700
-	0    -1   -1   0
-$EndComp
-Connection ~ 4750 1050
 $Comp
 L SW_PUSH SW1
@@
 	4150 1250 5350 1250
 $Comp
-L GND #PWR013
+L GND #PWR011
 U 1 1 5420D9A5
 P 6450 1250
-F 0 "#PWR013" H 6450 1250 30  0001 C CNN
+F 0 "#PWR011" H 6450 1250 30  0001 C CNN
 F 1 "GND" H 6450 1180 30  0001 C CNN
 F 2 "" H 6450 1250 60  0000 C CNN
@@
 L stm32f303x U1
 U 1 1 5420ED70
-P 3150 2300
-F 0 "U1" H 3150 4250 60  0000 C CNN
-F 1 "stm32f303x" H 3150 900 60  0000 C CNN
-F 2 "lqfp48:LQFP48" H 3150 2300 60  0001 C CNN
-F 3 "" H 3150 2300 60  0000 C CNN
-	1    3150 2300
+P 3050 2850
+F 0 "U1" H 3050 4800 60  0000 C CNN
+F 1 "stm32f303x" H 3050 1450 60  0000 C CNN
+F 2 "lqfp48:LQFP48" H 3050 2850 60  0001 C CNN
+F 3 "" H 3050 2850 60  0000 C CNN
+	1    3050 2850
 	1    0    0    -1
 $EndComp
 NoConn ~ 1950 3850
 NoConn ~ 1950 4250
-Wire Wire Line
-	1700 3000 1950 3000
-Wire Wire Line
-	1950 3600 1700 3600
-Wire Wire Line
-	1200 4800 1350 4800
 $Comp
 L TLV702xx U2
@@
 F 0 "U2" H 4200 6954 60  0000 C CNN
 F 1 "TLV702xx" H 4050 7350 60  0000 C CNN
-F 2 "SMD_Packages:SOT-23-5" H 4050 7150 60  0001 C CNN
+F 2 "SOT23-5:SOT23-5" H 4050 7150 60  0001 C CNN
 F 3 "" H 4050 7150 60  0000 C CNN
 	1    4050 7150
@@
 $EndComp
 Wire Wire Line
-	3550 7200 3650 7200
+	3450 7200 3650 7200
 Wire Wire Line
 	3050 7200 3050 7100
@@
 $EndComp
 $Comp
-L PWR_FLAG #FLG014
+L PWR_FLAG #FLG012
 U 1 1 54232740
 P 1100 1700
-F 0 "#FLG014" H 1100 1795 30  0001 C CNN
+F 0 "#FLG012" H 1100 1795 30  0001 C CNN
 F 1 "PWR_FLAG" H 1100 1880 30  0000 C CNN
 F 2 "" H 1100 1700 60  0000 C CNN
@@
 Connection ~ 1100 1700
 Wire Wire Line
-	1350 2750 1200 2750
+	1200 2750 1450 2750
 $Comp
 L R R5
@@
 	4150 2750 4350 2750
 Wire Wire Line
-	4750 2750 4900 2750
+	4750 2750 5000 2750
 Wire Wire Line
 	4150 2850 4350 2850
 Wire Wire Line
-	4750 2850 4900 2850
+	4750 2850 5000 2850
 Wire Wire Line
 	5400 2750 5400 2850
 $Comp
-L GND #PWR015
+L GND #PWR013
 U 1 1 54316E51
-P 5500 2850
-F 0 "#PWR015" H 5500 2850 30  0001 C CNN
-F 1 "GND" H 5500 2780 30  0001 C CNN
-F 2 "" H 5500 2850 60  0000 C CNN
-F 3 "" H 5500 2850 60  0000 C CNN
-	1    5500 2850
+P 5450 2850
+F 0 "#PWR013" H 5450 2850 30  0001 C CNN
+F 1 "GND" H 5450 2780 30  0001 C CNN
+F 2 "" H 5450 2850 60  0000 C CNN
+F 3 "" H 5450 2850 60  0000 C CNN
+	1    5450 2850
 	0    -1   -1   0
 $EndComp
 Wire Wire Line
-	5400 2850 5500 2850
+	5300 2850 5450 2850
 Connection ~ 5400 2850
 Wire Wire Line
-	5100 2200 5650 2200
+	5100 2200 5700 2200
 $Comp
 L TESTPOINT U4
@@
 $EndComp
 $Comp
-L GND #PWR018
+L GND #PWR014
 U 1 1 5431DFE3
 P 4650 3650
-F 0 "#PWR018" H 4650 3650 30  0001 C CNN
+F 0 "#PWR014" H 4650 3650 30  0001 C CNN
 F 1 "GND" H 4650 3580 30  0001 C CNN
 F 2 "" H 4650 3650 60  0000 C CNN
@@
 	5950 1250 5950 750
 $Comp
-L VDD #PWR020
+L VDD #PWR015
 U 1 1 5431FA98
 P 1200 2750
-F 0 "#PWR020" H 1200 2850 30  0001 C CNN
+F 0 "#PWR015" H 1200 2850 30  0001 C CNN
 F 1 "VDD" H 1200 2860 30  0000 C CNN
 F 2 "" H 1200 2750 60  0000 C CNN
@@
 	5100 1650 5100 2200
 Wire Wire Line
-	1350 2650 900  2650
+	900  2650 1450 2650
 Wire Wire Line
 	900  2650 900  2500
 Connection ~ 900  2500
 Wire Wire Line
-	5600 2100 5650 2100
+	5600 2100 5700 2100
 Text GLabel 5550 2000 0    60   Output ~ 0
 VCC5V
 Wire Wire Line
-	5650 2000 5550 2000
+	5550 2000 5700 2000
+Wire Wire Line
+	1100 2100 1100 2150
+Wire Wire Line
+	1300 2100 1300 2150
+Wire Wire Line
+	1100 2450 1100 2500
+Wire Wire Line
+	1300 2500 1300 2450
+Wire Wire Line
+	5300 2750 5400 2750
+$Comp
+L CONN_01X03 P2
+U 1 1 55590810
+P 5900 2100
+F 0 "P2" H 5900 2300 50  0000 C CNN
+F 1 "CONN_01X03" V 6000 2100 50  0000 C CNN
+F 2 "synic:jst-3-pth-ra" H 5900 2100 60  0001 C CNN
+F 3 "" H 5900 2100 60  0000 C CNN
+	1    5900 2100
+	1    0    0    -1
+$EndComp
+$Comp
+L Battery BT1
+U 1 1 55590E88
+P 1700 4800
+F 0 "BT1" H 1800 4850 50  0000 L CNN
+F 1 "3v" H 1800 4750 50  0000 L CNN
+F 2 "synicpretty:BK-755_12mm_coincell" V 1700 4840 60  0001 C CNN
+F 3 "" V 1700 4840 60  0000 C CNN
+	1    1700 4800
+	0    1    1    0
+$EndComp
+Wire Wire Line
+	1450 4800 1550 4800
+Wire Wire Line
+	1950 4800 1850 4800
+$Comp
+L Crystal_Small Y1
+U 1 1 5559168C
+P 1700 3300
+F 0 "Y1" H 1700 3400 50  0000 C CNN
+F 1 "32.768 KHz" H 1700 3200 50  0000 C CNN
+F 2 "synic:2_SMD_CRYSTAL_3.2x1.5" H 1700 3300 60  0001 C CNN
+F 3 "" H 1700 3300 60  0000 C CNN
+	1    1700 3300
+	0    1    1    0
+$EndComp
+Wire Wire Line
+	1700 3200 1700 3100
+Wire Wire Line
+	1700 3100 1950 3100
+Wire Wire Line
+	1700 3400 1700 3500
+Wire Wire Line
+	1700 3500 1950 3500
+NoConn ~ 4150 1050
+Wire Wire Line
+	2650 6300 2650 6350
+Wire Wire Line
+	3050 7200 3150 7200
+Wire Wire Line
+	2700 7150 2700 7100
+Wire Wire Line
+	2700 7450 2700 7500
+Wire Wire Line
+	4650 7450 4650 7500
+Wire Wire Line
+	4650 7100 4650 7150
+Wire Wire Line
+	1100 1300 1100 1250
+Wire Wire Line
+	1300 1300 1300 1250
+Wire Wire Line
+	1500 1300 1500 1250
+Wire Wire Line
+	1700 1300 1700 1250
+Wire Wire Line
+	1700 1600 1700 1650
+Wire Wire Line
+	1500 1600 1500 1650
+Wire Wire Line
+	1300 1600 1300 1650
 $EndSCHEMATC

Commit message: updating board
Parts:
- added U?: TXS0101, symbol TXS0101
Connections:
- wire segments 81 -> 94
Changed lines of the file:
@@
 L GND #PWR010
 U 1 1 5420B549
-P 5600 2100
-F 0 "#PWR010" H 5600 2100 30  0001 C CNN
-F 1 "GND" H 5600 2030 30  0001 C CNN
-F 2 "" H 5600 2100 60  0000 C CNN
-F 3 "" H 5600 2100 60  0000 C CNN
-	1    5600 2100
+P 5450 6350
+F 0 "#PWR010" H 5450 6350 30  0001 C CNN
+F 1 "GND" H 5450 6280 30  0001 C CNN
+F 2 "" H 5450 6350 60  0000 C CNN
+F 3 "" H 5450 6350 60  0000 C CNN
+	1    5450 6350
 	0    1    1    0
 $EndComp
@@
 Connection ~ 2700 7100
 Wire Wire Line
-	2350 6300 2350 7100
+	2350 6100 2350 7100
 Wire Wire Line
 	1450 7500 5150 7500
@@
 	5300 2850 5450 2850
 Connection ~ 5400 2850
-Wire Wire Line
-	5100 2200 5700 2200
 $Comp
 L TESTPOINT U4
 U 1 1 5431DE36
-P 5900 2950
-F 0 "U4" H 5900 2850 60  0000 C CNN
-F 1 "NEO" H 5900 3150 60  0000 C CNN
-F 2 "synicpretty:TESTPOINT" H 6000 2950 60  0001 C CNN
-F 3 "" H 6000 2950 60  0000 C CNN
-	1    5900 2950
-	1    0    0    -1
-$EndComp
-Wire Wire Line
-	5600 2900 5600 2200
-Connection ~ 5600 2200
+P 5900 6850
+F 0 "U4" H 5900 6750 60  0000 C CNN
+F 1 "NEO" H 5900 7050 60  0000 C CNN
+F 2 "synicpretty:TESTPOINT" H 6000 6850 60  0001 C CNN
+F 3 "" H 6000 6850 60  0000 C CNN
+	1    5900 6850
+	1    0    0    -1
+$EndComp
 $Comp
 L TESTPOINT U5
@@
 NoConn ~ 4150 2050
 Wire Wire Line
-	4150 1650 5100 1650
-Wire Wire Line
-	5100 1650 5100 2200
+	4150 1650 5700 1650
 Wire Wire Line
 	900  2650 1450 2650
@@
 	900  2650 900  2500
 Connection ~ 900  2500
-Wire Wire Line
-	5600 2100 5700 2100
-Text GLabel 5550 2000 0    60   Output ~ 0
+Text GLabel 5400 6250 0    60   Output ~ 0
 VCC5V
-Wire Wire Line
-	5550 2000 5700 2000
 Wire Wire Line
 	1100 2100 1100 2150
@@
 L CONN_01X03 P2
 U 1 1 55590810
-P 5900 2100
-F 0 "P2" H 5900 2300 50  0000 C CNN
-F 1 "CONN_01X03" V 6000 2100 50  0000 C CNN
-F 2 "synic:jst-3-pth-ra" H 5900 2100 60  0001 C CNN
-F 3 "" H 5900 2100 60  0000 C CNN
-	1    5900 2100
+P 5800 6350
+F 0 "P2" H 5800 6550 50  0000 C CNN
+F 1 "CONN_01X03" V 5900 6350 50  0000 C CNN
+F 2 "synic:jst-3-pth-ra" H 5800 6350 60  0001 C CNN
+F 3 "" H 5800 6350 60  0000 C CNN
+	1    5800 6350
 	1    0    0    -1
 $EndComp
@@
 Wire Wire Line
 	1300 1600 1300 1650
+$Comp
+L TXS0101 U?
+U 1 1 555909CF
+P 4250 6350
+F 0 "U?" H 4250 6050 60  0000 C CNN
+F 1 "TXS0101" H 4250 6550 60  0000 C CNN
+F 2 "" H 4250 6350 60  0000 C CNN
+F 3 "" H 4250 6350 60  0000 C CNN
+	1    4250 6350
+	1    0    0    -1
+$EndComp
+Wire Wire Line
+	3850 6300 3650 6300
+Wire Wire Line
+	3650 6300 3650 6850
+Wire Wire Line
+	3650 6850 4850 6850
+Wire Wire Line
+	4850 6400 4850 7100
+Connection ~ 4850 7100
+Wire Wire Line
+	4650 6300 4650 6100
+Wire Wire Line
+	4650 6100 2350 6100
+Connection ~ 2350 6300
+$Comp
+L GND #PWR?
+U 1 1 55590D84
+P 3800 6400
+F 0 "#PWR?" H 3800 6400 30  0001 C CNN
+F 1 "GND" H 3800 6330 30  0001 C CNN
+F 2 "" H 3800 6400 60  0000 C CNN
+F 3 "" H 3800 6400 60  0000 C CNN
+	1    3800 6400
+	0    1    1    0
+$EndComp
+Wire Wire Line
+	3800 6400 3850 6400
+Wire Wire Line
+	4850 6400 4650 6400
+Connection ~ 4850 6850
+Wire Wire Line
+	5600 6450 5600 6800
+Wire Wire Line
+	5450 6350 5600 6350
+Wire Wire Line
+	5400 6250 5600 6250
+Wire Wire Line
+	5700 1650 5700 5600
+Wire Wire Line
+	5700 5600 3550 5600
+Wire Wire Line
+	3550 5600 3550 6500
+Wire Wire Line
+	3550 6500 3850 6500
+Wire Wire Line
+	4650 6500 5450 6500
+Wire Wire Line
+	5450 6500 5450 6450
+Wire Wire Line
+	5450 6450 5600 6450
 $EndSCHEMATC

Commit message: woot
Parts:
- U3: renamed from U?; footprint (none) -> Housings_SOT-23_SOT-143_TSOT-6:SOT-23-6
Changed lines of the file:
@@
 	1300 1600 1300 1650
 $Comp
-L TXS0101 U?
+L TXS0101 U3
 U 1 1 555909CF
 P 4250 6350
-F 0 "U?" H 4250 6050 60  0000 C CNN
+F 0 "U3" H 4250 6050 60  0000 C CNN
 F 1 "TXS0101" H 4250 6550 60  0000 C CNN
-F 2 "" H 4250 6350 60  0000 C CNN
+F 2 "Housings_SOT-23_SOT-143_TSOT-6:SOT-23-6" H 4250 6350 60  0001 C CNN
 F 3 "" H 4250 6350 60  0000 C CNN
 	1    4250 6350
@@
 Connection ~ 2350 6300
 $Comp
-L GND #PWR?
+L GND #PWR016
 U 1 1 55590D84
 P 3800 6400
-F 0 "#PWR?" H 3800 6400 30  0001 C CNN
+F 0 "#PWR016" H 3800 6400 30  0001 C CNN
 F 1 "GND" H 3800 6330 30  0001 C CNN
 F 2 "" H 3800 6400 60  0000 C CNN
